Commit message: Modified r1d1_description with working RGBD camera

File: r1d1_description/urdf/lidar.xacro (robot description, xacro)
@@ -1,54 +1,55 @@
 <?xml version="1.0"?>
 <robot xmlns:xacro="http://www.ros.org/wiki/xacro" >
-    <joint name="laser_joint" type="fixed">
-        <parent link="base_link"/>
-        <child link="laser_frame"/>
-        <origin xyz="0.20 0 0.24" rpy="0 0 0"/>
-    </joint>
-    <link name="laser_frame">
-        <visual>
-            <geometry>
-                <cylinder radius="0.05" length="0.04"/>
-            </geometry>
-            <material name="red">
-            <color rgba="1 0 0 1.000"/>
-            </material>
-        </visual>
-        <collision>
-            <geometry>
-                <cylinder radius="0.05" length="0.04"/>
-            </geometry>
-        </collision>
-        <xacro:inertial_cylinder mass="0.1" length="0.04" radius="0.05">
-            <origin xyz="0 0 0" rpy="0 0 0"/>
-        </xacro:inertial_cylinder>
-    </link>
-    <gazebo reference="laser_frame">
-        <material>Gazebo/Red</material>
-        <sensor name="laser" type="ray">
-            <pose> 0 0 0 0 0 0 </pose>
-            <visualize>true</visualize>
-            <update_rate>10</update_rate>
-            <ray>
-                <scan>
-                    <horizontal>
-                        <samples>720</samples>
-                        <min_angle>-1.54</min_angle>
-                        <max_angle>1.54</max_angle>
-                    </horizontal>
-                </scan>
-                <range>
-                    <min>0.15</min>
-                    <max>12</max>
-                </range>
-            </ray>
-            <plugin name="laser_controller" filename="libgazebo_ros_ray_sensor.so">
-                <ros>
-                    <argument>~--ros-args --remap ~/out:=/scan</argument>
-                </ros>
-                <output_type>sensor_msgs/LaserScan</output_type>
-                <frame_name>laser_frame</frame_name>
-            </plugin>
-        </sensor>
-    </gazebo>
+<!--This file has added code for lidar. Uncomment the include line in r1d1.xacro to include lidar-->
+  <joint name="Rigid 46" type="fixed">
+    <origin xyz="0.0 -0.123483 0.155" rpy="0 0 0"/>
+    <parent link="base_link"/>
+    <child link="lidar_1"/>
+  </joint>
+  <link name="lidar_1">
+    <inertial>
+      <origin xyz="-3.8657673471382324e-17 -4.13193513695842e-07 0.015000000000000013" rpy="0 0 0"/>
+      <mass value="0.6616194128460102"/>
+      <inertia ixx="0.00048" iyy="0.00048" izz="0.00086" ixy="0.0" iyz="-0.0" ixz="0.0"/>
+    </inertial>
+    <visual>
+      <origin xyz="0.0 0.123483 -0.155" rpy="0 0 0"/>
+      <geometry>
+        <mesh filename="file://$(find r1d1_description)/meshes/lidar_1.stl" scale="0.001 0.001 0.001"/>
+      </geometry>
+      <material name="silver"/>
+    </visual>
+    <collision>
+      <origin xyz="0.0 0.123483 -0.155" rpy="0 0 0"/>
+      <geometry>
+        <mesh filename="file://$(find r1d1_description)/meshes/lidar_1.stl" scale="0.001 0.001 0.001"/>
+      </geometry>
+    </collision>
+  </link>
+  <gazebo reference="lidar_1">
+    <material>Gazebo/Red</material>
+    <sensor name="gpu_lidar" type="gpu_lidar">
+      <lidar>
+        <scan>
+          <horizontal>
+            <samples>720</samples>
+            <min_angle>-1.54</min_angle>
+            <max_angle>1.54</max_angle>
+          </horizontal>
+        </scan>
+        <range>
+          <min>0.15</min>
+          <max>12</max>
+        </range>
+      </lidar>
+      <alwaysOn>true</alwaysOn>
+      <topic>lidar_data</topic>
+      <pose> 0 0 0 0 0 0 </pose>
+      <visualize>true</visualize>
+      <update_rate>10</update_rate>
+      <plugin filename="ignition-gazebo-sensors-system" name="gz::sim::systems::Sensors">
+        <render_engine>ogre2</render_engine>
+      </plugin>
+    </sensor>
+  </gazebo>
 </robot>

File: r1d1_description/urdf/r1d1.urdf (robot description, URDF)
Before this commit: robot r1d1, 16 links, 15 joints
Links:
- removed link arm_base_link_1
- removed link base_footprint
- removed link c1_1
- removed link c2_1
- removed link c3_1
- removed link c4_1
- removed link forearm_Link_1
- removed link linear_1
- removed link shoulder_Link_1
- removed link upperarm_Link_1
- removed link wrist1_Link_1
- removed link wrist2_Link_1
- removed link wrist3_Link_1
- added link amr_c2_1, mass 0.8336850329541245; collision mesh filename=file:///home/ishan/OpenDroids_ws/install/r1d1_description/s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 scale=0.001 0.001 0.001; visual mesh filename=file:///home/ishan/OpenDroids_ws/install/r1d1_description/s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 scale=0.001 0.001 0.001
- added link amr_c3_1, mass 2.940490372828695; collision mesh filename=file:///home/ishan/OpenDroids_ws/install/r1d1_description/s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 scale=0.001 0.001 0.001; visual mesh filename=file:///home/ishan/OpenDroids_ws/install/r1d1_description/s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 scale=0.001 0.001 0.001
- added link arm_c1_1, mass 0.3077654114507175; collision mesh filename=file:///home/ishan/OpenDroids_ws/install/r1d1_description/s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 scale=0.001 0.001 0.001; visual mesh filename=file:///home/ishan/OpenDroids_ws/install/r1d1_description/s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 scale=0.001 0.001 0.001
- added link arm_c4_1, mass 1.9148915468217087; collision mesh filename=file:///home/ishan/OpenDroids_ws/install/r1d1_description/s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 scale=0.001 0.001 0.001; visual mesh filename=file:///home/ishan/OpenDroids_ws/install/r1d1_description/s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 scale=0.001 0.001 0.001
- added link arm_c5_1, mass 0.7917902286710067; collision mesh filename=file:///home/ishan/OpenDroids_ws/install/r1d1_description/s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 scale=0.001 0.001 0.001; visual mesh filename=file:///home/ishan/OpenDroids_ws/install/r1d1_description/s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 scale=0.001 0.001 0.001
- added link arm_c6_1, mass 0.6685877298515001; collision mesh filename=file:///home/ishan/OpenDroids_ws/install/r1d1_description/s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 scale=0.001 0.001 0.001; visual mesh filename=file:///home/ishan/OpenDroids_ws/install/r1d1_description/s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 scale=0.001 0.001 0.001
- added link arm_c7_1, mass 0.21151566499231975; collision mesh filename=file:///home/ishan/OpenDroids_ws/install/r1d1_description/s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 scale=0.001 0.001 0.001; visual mesh filename=file:///home/ishan/OpenDroids_ws/install/r1d1_description/s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 scale=0.001 0.001 0.001
- added link camera_1, mass 0.05166258768470149; collision mesh filename=file:///home/ishan/OpenDroids_ws/install/r1d1_description/s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 scale=0.001 0.001 0.001; visual mesh filename=file:///home/ishan/OpenDroids_ws/install/r1d1_description/s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 scale=0.001 0.001 0.001
- added link caster_1_1, mass 0.18492935556768103; collision mesh filename=file:///home/ishan/OpenDroids_ws/install/r1d1_description/s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 scale=0.001 0.001 0.001; visual mesh filename=file:///home/ishan/OpenDroids_ws/install/r1d1_description/s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 scale=0.001 0.001 0.001
- added link gripper_base_1, mass 0.7474580686995151; collision mesh filename=file:///home/ishan/OpenDroids_ws/install/r1d1_description/s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 scale=0.001 0.001 0.001; visual mesh filename=file:///home/ishan/OpenDroids_ws/install/r1d1_description/s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 scale=0.001 0.001 0.001
- added link gripper_finger2_1, mass 0.016384204166531253; collision mesh filename=file:///home/ishan/OpenDroids_ws/install/r1d1_description/s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 scale=0.001 0.001 0.001; visual mesh filename=file:///home/ishan/OpenDroids_ws/install/r1d1_description/s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 scale=0.001 0.001 0.001
- added link gripper_finger_1, mass 0.016384204166531253; collision mesh filename=file:///home/ishan/OpenDroids_ws/install/r1d1_description/s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 scale=0.001 0.001 0.001; visual mesh filename=file:///home/ishan/OpenDroids_ws/install/r1d1_description/s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 scale=0.001 0.001 0.001
- added link mount_v1_1, mass 37.46152841680288; collision mesh filename=file:///home/ishan/OpenDroids_ws/install/r1d1_description/s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 scale=0.001 0.001 0.001; visual mesh filename=file:///home/ishan/OpenDroids_ws/install/r1d1_description/s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 scale=0.001 0.001 0.001
- added link screen_v1_1, mass 1.3238858059375562; collision mesh filename=file:///home/ishan/OpenDroids_ws/install/r1d1_description/s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 scale=0.001 0.001 0.001; visual mesh filename=file:///home/ishan/OpenDroids_ws/install/r1d1_description/s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 scale=0.001 0.001 0.001
- added link slider_1, mass 0.43604999999999994; collision mesh filename=file:///home/ishan/OpenDroids_ws/install/r1d1_description/s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 scale=0.001 0.001 0.001; visual mesh filename=file:///home/ishan/OpenDroids_ws/install/r1d1_description/s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 scale=0.001 0.001 0.001
- added link vertical_v1_1, mass 24.32699999999999; collision mesh filename=file:///home/ishan/OpenDroids_ws/install/r1d1_description/s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 scale=0.001 0.001 0.001; visual mesh filename=file:///home/ishan/OpenDroids_ws/install/r1d1_description/s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 scale=0.001 0.001 0.001
- link base_link: mass 55.61253674388458 -> 36.898914712235424; geometry collision mesh filename=file:///home/ishan/OpenDroids_ws/install/r1d1_description/s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 scale=0.001 0.001 0.001; visual mesh filename=file:///home/ishan/OpenDroids_ws/install/r1d1_description/s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 scale=0.001 0.001 0.001
- link left_wheel_1: mass 3.081377574152813 -> 1.2020197871482743; geometry collision mesh filename=file:///home/ishan/OpenDroids_ws/install/r1d1_description/s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 scale=0.001 0.001 0.001; visual mesh filename=file:///home/ishan/OpenDroids_ws/install/r1d1_description/s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 scale=0.001 0.001 0.001
- link right_wheel_1: mass 3.0813775741527913 -> 1.2020197871482743; geometry collision mesh filename=file:///home/ishan/OpenDroids_ws/install/r1d1_description/s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 scale=0.001 0.001 0.001; visual mesh filename=file:///home/ishan/OpenDroids_ws/install/r1d1_description/s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 scale=0.001 0.001 0.001
Joints:
- removed joint arm_fixed_joint
- removed joint base_footprint_joint
- removed joint castor_1
- removed joint castor_2
- removed joint castor_3
- removed joint castor_4
- removed joint forearm_joint
- removed joint shoulder_joint
- removed joint slider
- removed joint upperarm_joint
- removed joint wrist_joint_1
- removed joint wrist_joint_2
- removed joint wrist_joint_3
- added joint Revolute 35: type continuous, parent arm_c1_1, child amr_c2_1, origin xyz=0.0 -0.0798 0.0 rpy=0 0 0, axis 0.0 -1.0 -0.0
- added joint Revolute 38: type continuous, parent amr_c3_1, child arm_c4_1, origin xyz=0.197628 0.0 0.19835 rpy=0 0 0, axis 0.708394 0.0 -0.705817
- added joint Revolute 39: type continuous, parent arm_c4_1, child arm_c5_1, origin xyz=0.168837 0.0 0.170587 rpy=0 0 0, axis -0.708394 -0.0 0.705817
- added joint Revolute 40: type continuous, parent arm_c5_1, child arm_c6_1, origin xyz=0.07106 -0.009116 0.00218 rpy=0 0 0, axis -0.695094 0.173648 -0.697632
- added joint Revolute 41: type continuous, parent amr_c2_1, child amr_c3_1, origin xyz=0.038112 -0.06 -0.037973 rpy=0 0 0, axis 0.708394 0.0 -0.705817
- added joint Revolute 42: type continuous, parent arm_c6_1, child arm_c7_1, origin xyz=0.074299 -0.008474 -0.006187 rpy=0 0 0, axis 0.708394 0.0 -0.705817
- added joint Rigid 21: type fixed, parent base_link, child mount_v1_1, origin xyz=0.0 0.0 0.28 rpy=0 0 0
- added joint Rigid 23: type fixed, parent mount_v1_1, child vertical_v1_1, origin xyz=-0.300276 0.208406 2.495761 rpy=0 0 0
- added joint Rigid 31: type fixed, parent vertical_v1_1, child screen_v1_1, origin xyz=0.300276 -0.123405 -0.990761 rpy=0 0 0
- added joint Rigid 34: type fixed, parent slider_1, child arm_c1_1, origin xyz=0.0 -0.005 0.0 rpy=0 0 0
- added joint Rigid 43: type fixed, parent arm_c7_1, child gripper_base_1, origin xyz=0.030461 0.0 -0.03035 rpy=0 0 0
- added joint Rigid 45: type fixed, parent screen_v1_1, child camera_1, origin xyz=0.0 -0.117 0.0525 rpy=0 0 0
- added joint Rigid 7: type fixed, parent base_link, child caster_1_1, origin xyz=0.0 0.0 0.0 rpy=0 0 0
- added joint Slider 29: type prismatic, parent gripper_base_1, child gripper_finger_1, origin xyz=1.429463 0.07146 -0.432363 rpy=0 0 0, axis 0.695094 -0.173648 0.697632, limit lower=0.0055 upper=0.045 effort=100 velocity=100
- added joint Slider 30: type prismatic, parent gripper_base_1, child gripper_finger2_1, origin xyz=1.429463 0.07146 -0.432363 rpy=0 0 0, axis 0.695094 -0.173648 0.697632, limit lower=-0.04 upper=-0.0005 effort=100 velocity=100
- added joint Slider 33: type prismatic, parent vertical_v1_1, child slider_1, origin xyz=0.300276 -0.213405 -1.740761 rpy=0 0 0, axis 0.0 -0.0 1.0, limit lower=-0.64 upper=0.64 effort=100 velocity=100
- joint left_wheel_joint: axis -0.0 1.0 0.0 -> -1.0 0.0 0.0; origin xyz=0.0 0.105 0.085 rpy=0 0 0 -> xyz=0.125905 0.011214 0.01 rpy=0 0 0
- joint right_wheel_joint: axis 0.0 1.0 -0.0 -> 1.0 -0.0 0.0; origin xyz=0.0 -0.105 0.085 rpy=0 0 0 -> xyz=-0.125905 0.011214 0.01 rpy=0 0 0
