Commit message: divide the slider & arm group

File: r1d1_description/urdf/ros2_control.xacro (robot description, xacro)
@@ -37,13 +37,9 @@
         </hardware>
         <joint name="slider">
-            <command_interface name="position">
-            <param name="min">-0.7</param>
-            <param name="max">0.5</param>
-            </command_interface>
+            <command_interface name="position"/>
             <state_interface name="position">
-            <param name="initial_value">0.0</param>
+                <param name="initial_value">0.3</param>
             </state_interface>
             <state_interface name="velocity"/>
-            <state_interface name="effort"/>
         </joint>
         <joint name="castor_1">

File: r1d1_moveit2_config/config/r1d1.ros2_control.xacro (robot description, xacro)
@@ -8,11 +8,4 @@
                 <plugin>mock_components/GenericSystem</plugin>
             </hardware>
-            <joint name="slider">
-                <command_interface name="position"/>
-                <state_interface name="position">
-                  <param name="initial_value">${initial_positions['slider']}</param>
-                </state_interface>
-                <state_interface name="velocity"/>
-            </joint>
             <joint name="shoulder_joint">
                 <command_interface name="position"/>
@@ -57,4 +50,11 @@
                 <state_interface name="velocity"/>
             </joint>
+            <joint name="slider">
+                <command_interface name="position"/>
+                <state_interface name="position">
+                  <param name="initial_value">${initial_positions['slider']}</param>
+                </state_interface>
+                <state_interface name="velocity"/>
+            </joint>
         </ros2_control>
     </xacro:macro>

Commit message: change moveit config

File: r1d1_description/urdf/ros2_control.xacro (robot description, xacro)
@@ -97,4 +97,18 @@
             <state_interface name="effort"/>
         </joint>
+        <joint name="Slider 29">
+            <command_interface name="position"/>
+            <state_interface name="position">
+                <param name="initial_value">0.0081</param>
+            </state_interface>
+            <state_interface name="velocity"/>
+        </joint>
+        <joint name="Slider 30">
+            <command_interface name="position"/>
+            <state_interface name="position">
+                <param name="initial_value">-0.0040</param>
+            </state_interface>
+            <state_interface name="velocity"/>
+        </joint>
         <joint name="left_wheel_joint">
                 <command_interface name="velocity">

File: r1d1_moveit2_config/config/r1d1.ros2_control.xacro (robot description, xacro)
@@ -8,50 +8,64 @@
                 <plugin>mock_components/GenericSystem</plugin>
             </hardware>
-            <joint name="shoulder_joint">
+            <joint name="Revolute 35">
                 <command_interface name="position"/>
                 <state_interface name="position">
-                  <param name="initial_value">${initial_positions['shoulder_joint']}</param>
+                  <param name="initial_value">${initial_positions['Revolute 35']}</param>
                 </state_interface>
                 <state_interface name="velocity"/>
             </joint>
-            <joint name="upperarm_joint">
+            <joint name="Revolute 41">
                 <command_interface name="position"/>
                 <state_interface name="position">
-                  <param name="initial_value">${initial_positions['upperarm_joint']}</param>
+                  <param name="initial_value">${initial_positions['Revolute 41']}</param>
                 </state_interface>
                 <state_interface name="velocity"/>
             </joint>
-            <joint name="forearm_joint">
+            <joint name="Revolute 38">
                 <command_interface name="position"/>
                 <state_interface name="position">
-                  <param name="initial_value">${initial_positions['forearm_joint']}</param>
+                  <param name="initial_value">${initial_positions['Revolute 38']}</param>
                 </state_interface>
                 <state_interface name="velocity"/>
             </joint>
-            <joint name="wrist_joint_1">
+            <joint name="Revolute 39">
                 <command_interface name="position"/>
                 <state_interface name="position">
-                  <param name="initial_value">${initial_positions['wrist_joint_1']}</param>
+                  <param name="initial_value">${initial_positions['Revolute 39']}</param>
                 </state_interface>
                 <state_interface name="velocity"/>
             </joint>
-            <joint name="wrist_joint_2">
+            <joint name="Revolute 40">
                 <command_interface name="position"/>
                 <state_interface name="position">
-                  <param name="initial_value">${initial_positions['wrist_joint_2']}</param>
+                  <param name="initial_value">${initial_positions['Revolute 40']}</param>
                 </state_interface>
                 <state_interface name="velocity"/>
             </joint>
-            <joint name="wrist_joint_3">
+            <joint name="Revolute 42">
                 <command_interface name="position"/>
                 <state_interface name="position">
-                  <param name="initial_value">${initial_positions['wrist_joint_3']}</param>
+                  <param name="initial_value">${initial_positions['Revolute 42']}</param>
                 </state_interface>
                 <state_interface name="velocity"/>
             </joint>
-            <joint name="slider">
+            <joint name="Slider 33">
                 <command_interface name="position"/>
                 <state_interface name="position">
-                  <param name="initial_value">${initial_positions['slider']}</param>
+                  <param name="initial_value">${initial_positions['Slider 33']}</param>
+                </state_interface>
+                <state_interface name="velocity"/>
+            </joint>
+            <joint name="Slider 29">
+                <command_interface name="position"/>
+                <state_interface name="position">
+                  <param name="initial_value">${initial_positions['Slider 29']}</param>
+                </state_interface>
+                <state_interface name="velocity"/>
+            </joint>
+            <joint name="Slider 30">
+                <command_interface name="position"/>
+                <state_interface name="position">
+                  <param name="initial_value">${initial_positions['Slider 30']}</param>
                 </state_interface>
                 <state_interface name="velocity"/>
