Commit message: Add files via upload

File: r1d1_description/urdf/r1d1.urdf (robot description, URDF)
Before this commit: robot r1d1, 19 links, 18 joints
Links:
- added link lidar_1, mass 0.6616194128460102; collision mesh filename=file:///home/ishan/OpenDroids_ws/install/r1d1_description/s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 scale=0.001 0.001 0.001; visual mesh filename=file:///home/ishan/OpenDroids_ws/install/r1d1_description/s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 scale=0.001 0.001 0.001
Joints:
- added joint Rigid 46: type fixed, parent base_link, child lidar_1, origin xyz=0.0 -0.123483 0.155 rpy=0 0 0
- joint Rigid 45: axis (none) -> 0 0 1; limit (none) -> lower=0 upper=0 effort=0 velocity=0; type fixed -> revolute

File: r1d1_description/urdf/r1d1.xacro (robot description, xacro)
@@ -1,471 +1,492 @@
 <?xml version="1.0" ?>
-<robot name="r1d1" xmlns:xacro="http://www.ros.org/wiki/xacro">
-<xacro:include filename="$(find r1d1_description)/urdf/materials.xacro" />
-<!--<xacro:include filename="$(find r1d1_description)/urdf/lidar.xacro" />-->
-<xacro:include filename="$(find r1d1_description)/urdf/rgbd_camera.xacro" />
-<xacro:include filename="$(find r1d1_description)/urdf/r1d1.trans" />
-<xacro:include filename="$(find r1d1_description)/urdf/r1d1.gazebo" />
-<link name="base_link">
-  <inertial>
-    <origin xyz="1.1547257273897802e-06 -0.007635347278315616 0.15138662427903304" rpy="0 0 0"/>
-    <mass value="36.898914712235424"/>
-    <inertia ixx="0.87793" iyy="0.993842" izz="1.325469" ixy="2.9e-05" iyz="-0.00262" ixz="9e-06"/>
-  </inertial>
-  <visual>
-    <origin xyz="0 0 0" rpy="0 0 0"/>
-    <geometry>
-      <mesh filename="file://$(find r1d1_description)/meshes/base_link.stl" scale="0.001 0.001 0.001"/>
-    </geometry>
-    <material name="silver"/>
-  </visual>
-  <collision>
-    <origin xyz="0 0 0" rpy="0 0 0"/>
-    <geometry>
-      <mesh filename="file://$(find r1d1_description)/meshes/base_link.stl" scale="0.001 0.001 0.001"/>
-    </geometry>
-  </collision>
-</link>
-<link name="left_wheel_1">
-  <inertial>
-    <origin xyz="0.03933261352596262 -3.102141997377017e-07 3.896188927043909e-15" rpy="0 0 0"/>
-    <mass value="1.2020197871482743"/>
-    <inertia ixx="0.003741" iyy="0.002176" izz="0.002176" ixy="-0.0" iyz="0.0" ixz="0.0"/>
-  </inertial>
-  <visual>
-    <origin xyz="-0.125905 -0.011214 -0.01" rpy="0 0 0"/>
-    <geometry>
-      <mesh filename="file://$(find r1d1_description)/meshes/left_wheel_1.stl" scale="0.001 0.001 0.001"/>
-    </geometry>
-    <material name="silver"/>
-  </visual>
-  <collision>
-    <origin xyz="-0.125905 -0.011214 -0.01" rpy="0 0 0"/>
-    <geometry>
-      <mesh filename="file://$(find r1d1_description)/meshes/left_wheel_1.stl" scale="0.001 0.001 0.001"/>
-    </geometry>
-  </collision>
-</link>
-<link name="right_wheel_1">
-  <inertial>
-    <origin xyz="-0.03933261352596262 1.2614637535327683e-06 3.896188927043909e-15" rpy="0 0 0"/>
-    <mass value="1.2020197871482743"/>
-    <inertia ixx="0.003741" iyy="0.002176" izz="0.002176" ixy="-0.0" iyz="-0.0" ixz="-0.0"/>
-  </inertial>
-  <visual>
-    <origin xyz="0.125905 -0.011214 -0.01" rpy="0 0 0"/>
-    <geometry>
-      <mesh filename="file://$(find r1d1_description)/meshes/right_wheel_1.stl" scale="0.001 0.001 0.001"/>
-    </geometry>
-    <material name="silver"/>
-  </visual>
-  <collision>
-    <origin xyz="0.125905 -0.011214 -0.01" rpy="0 0 0"/>
-    <geometry>
-      <mesh filename="file://$(find r1d1_description)/meshes/right_wheel_1.stl" scale="0.001 0.001 0.001"/>
-    </geometry>
-  </collision>
-</link>
-<link name="caster_1_1">
-  <inertial>
-    <origin xyz="0.0749999955448851 0.17500002391840322 -0.037229533269406326" rpy="0 0 0"/>
-    <mass value="0.18492935556768103"/>
-    <inertia ixx="0.000111" iyy="9.7e-05" izz="8.2e-05" ixy="0.0" iyz="-0.0" ixz="0.0"/>
-  </inertial>
-  <visual>
-    <origin xyz="-0.0 -0.0 -0.0" rpy="0 0 0"/>
-    <geometry>
-      <mesh filename="file://$(find r1d1_description)/meshes/caster_1_1.stl" scale="0.001 0.001 0.001"/>
-    </geometry>
-    <material name="silver"/>
-  </visual>
-  <collision>
-    <origin xyz="-0.0 -0.0 -0.0" rpy="0 0 0"/>
-    <geometry>
-      <mesh filename="file://$(find r1d1_description)/meshes/caster_1_1.stl" scale="0.001 0.001 0.001"/>
-    </geometry>
-  </collision>
-</link>
-<link name="mount_v1_1">
-  <inertial>
-    <origin xyz="0.004699834778461813 0.06797243215558421 0.5691408369250166" rpy="0 0 0"/>
-    <mass value="37.46152841680288"/>
-    <inertia ixx="7.91068" iyy="8.256966" izz="0.734564" ixy="0.009948" iyz="-0.366828" ixz="-0.022667"/>
-  </inertial>
-  <visual>
-    <origin xyz="-0.0 -0.0 -0.28" rpy="0 0 0"/>
-    <geometry>
-      <mesh filename="file://$(find r1d1_description)/meshes/mount_v1_1.stl" scale="0.001 0.001 0.001"/>
-    </geometry>
-    <material name="silver"/>
-  </visual>
-  <collision>
-    <origin xyz="-0.0 -0.0 -0.28" rpy="0 0 0"/>
-    <geometry>
-      <mesh filename="file://$(find r1d1_description)/meshes/mount_v1_1.stl" scale="0.001 0.001 0.001"/>
-    </geometry>
-  </collision>
-</link>
-<link name="vertical_v1_1">
-  <inertial>
-    <origin xyz="0.300276 -0.16840510951680002 -1.74076100000007" rpy="0 0 0"/>
-    <mass value="24.32699999999999"/>
-    <inertia ixx="4.577733" iyy="4.6199" izz="0.075008" ixy="-0.0" iyz="0.0" ixz="-0.0"/>
-  </inertial>
-  <visual>
-    <origin xyz="0.300276 -0.208406 -2.775761" rpy="0 0 0"/>
-    <geometry>
-      <mesh filename="file://$(find r1d1_description)/meshes/vertical_v1_1.stl" scale="0.001 0.001 0.001"/>
-    </geometry>
-    <material name="silver"/>
-  </visual>
-  <collision>
-    <origin xyz="0.300276 -0.208406 -2.775761" rpy="0 0 0"/>
-    <geometry>
-      <mesh filename="file://$(find r1d1_description)/meshes/vertical_v1_1.stl" scale="0.001 0.001 0.001"/>
-    </geometry>
-  </collision>
-</link>
-<link name="gripper_finger_1">
-  <inertial>
-    <origin xyz="-1.2887005800870863 -0.07296498486252255 0.3041595690014297" rpy="0 0 0"/>
-    <mass value="0.016384204166531253"/>
-    <inertia ixx="7e-06" iyy="1e-05" izz="5e-06" ixy="-0.0" iyz="0.0" ixz="4e-06"/>
-  </inertial>
-  <visual>
-    <origin xyz="-2.00986 0.095929 -0.899244" rpy="0 0 0"/>
-    <geometry>
-      <mesh filename="file://$(find r1d1_description)/meshes/gripper_finger_1.stl" scale="0.001 0.001 0.001"/>
-    </geometry>
-    <material name="silver"/>
-  </visual>
-  <collision>
-    <origin xyz="-2.00986 0.095929 -0.899244" rpy="0 0 0"/>
-    <geometry>
-      <mesh filename="file://$(find r1d1_description)/meshes/gripper_finger_1.stl" scale="0.001 0.001 0.001"/>
-    </geometry>
-  </collision>
-</link>
-<link name="gripper_finger2_1">
-  <inertial>
-    <origin xyz="-1.3007475016955818 -0.06995542399105785 0.2920686540778593" rpy="0 0 0"/>
-    <mass value="0.016384204166531253"/>
-    <inertia ixx="5e-06" iyy="1e-05" izz="7e-06" ixy="0.0" iyz="-0.0" ixz="4e-06"/>
-  </inertial>
-  <visual>
-    <origin xyz="-2.00986 0.095929 -0.899244" rpy="0 0 0"/>
-    <geometry>
-      <mesh filename="file://$(find r1d1_description)/meshes/gripper_finger2_1.stl" scale="0.001 0.001 0.001"/>
-    </geometry>
-    <material name="silver"/>
-  </visual>
-  <collision>
-    <origin xyz="-2.00986 0.095929 -0.899244" rpy="0 0 0"/>
-    <geometry>
-      <mesh filename="file://$(find r1d1_description)/meshes/gripper_finger2_1.stl" scale="0.001 0.001 0.001"/>
-    </geometry>
-  </collision>
-</link>
-<link name="screen_v1_1">
-  <inertial>
-    <origin xyz="1.84011819724741e-11 -0.03889295266081586 0.11598843171162043" rpy="0 0 0"/>
-    <mass value="1.3238858059375562"/>
-    <inertia ixx="0.00685" iyy="0.008161" izz="0.003561" ixy="0.0" iyz="0.001577" ixz="0.0"/>
-  </inertial>
-  <visual>
-    <origin xyz="-0.0 -0.085001 -1.785" rpy="0 0 0"/>
-    <geometry>
-      <mesh filename="file://$(find r1d1_description)/meshes/screen_v1_1.stl" scale="0.001 0.001 0.001"/>
-    </geometry>
-    <material name="silver"/>
-  </visual>
-  <collision>
-    <origin xyz="-0.0 -0.085001 -1.785" rpy="0 0 0"/>
-    <geometry>
-      <mesh filename="file://$(find r1d1_description)/meshes/screen_v1_1.stl" scale="0.001 0.001 0.001"/>
-    </geometry>
-  </collision>
-</link>
-<link name="slider_1">
-  <inertial>
-    <origin xyz="-5.902504556725109e-18 -0.002500109516799993 -6.994405055138486e-14" rpy="0 0 0"/>
-    <mass value="0.43604999999999994"/>
-    <inertia ixx="0.001313" iyy="0.002362" izz="0.001051" ixy="0.0" iyz="0.0" ixz="-0.0"/>
-  </inertial>
-  <visual>
-    <origin xyz="0.0 0.004999 -1.035" rpy="0 0 0"/>
-    <geometry>
-      <mesh filename="file://$(find r1d1_description)/meshes/slider_1.stl" scale="0.001 0.001 0.001"/>
-    </geometry>
-    <material name="silver"/>
-  </visual>
-  <collision>
-    <origin xyz="0.0 0.004999 -1.035" rpy="0 0 0"/>
-    <geometry>
-      <mesh filename="file://$(find r1d1_description)/meshes/slider_1.stl" scale="0.001 0.001 0.001"/>
-    </geometry>
-  </collision>
-</link>
-<link name="arm_c1_1">
-  <inertial>
-    <origin xyz="-2.78263793284472e-05 -0.032527409110111094 -0.0006654684875286865" rpy="0 0 0"/>
-    <mass value="0.3077654114507175"/>
-    <inertia ixx="0.000539" iyy="0.000776" izz="0.000548" ixy="0.0" iyz="6e-06" ixz="0.0"/>
-  </inertial>
-  <visual>
-    <origin xyz="0.0 0.009999 -1.035" rpy="0 0 0"/>
-    <geometry>
-      <mesh filename="file://$(find r1d1_description)/meshes/arm_c1_1.stl" scale="0.001 0.001 0.001"/>
-    </geometry>
-    <material name="silver"/>
-  </visual>
-  <collision>
-    <origin xyz="0.0 0.009999 -1.035" rpy="0 0 0"/>
-    <geometry>
-      <mesh filename="file://$(find r1d1_description)/meshes/arm_c1_1.stl" scale="0.001 0.001 0.001"/>
-    </geometry>
-  </collision>
-</link>
-<link name="amr_c2_1">
-  <inertial>
-    <origin xyz="0.0017122003101182226 -0.05521343954562406 -0.0017056690936951835" rpy="0 0 0"/>
-    <mass value="0.8336850329541245"/>
-    <inertia ixx="0.001385" iyy="0.000909" izz="0.001385" ixy="9e-06" iyz="-9e-06" ixz="1.6e-05"/>
-  </inertial>
-  <visual>
-    <origin xyz="-0.0 0.089799 -1.035" rpy="0 0 0"/>
-    <geometry>
-      <mesh filename="file://$(find r1d1_description)/meshes/amr_c2_1.stl" scale="0.001 0.001 0.001"/>
-    </geometry>
-    <material name="silver"/>
-  </visual>
-  <collision>
-    <origin xyz="-0.0 0.089799 -1.035" rpy="0 0 0"/>
-    <geometry>
-      <mesh filename="file://$(find r1d1_description)/meshes/amr_c2_1.stl" scale="0.001 0.001 0.001"/>
-    </geometry>
-  </collision>
-</link>
-<link name="arm_c4_1">
-  <inertial>
-    <origin xyz="0.055635248736101484 -3.323298905510974e-08 0.12568017736494497" rpy="0 0 0"/>
-    <mass value="1.9148915468217087"/>
-    <inertia ixx="0.010371" iyy="0.017911" izz="0.00916" ixy="-0.0" iyz="-0.0" ixz="-0.007787"/>
-  </inertial>
-  <visual>
-    <origin xyz="-0.23574 0.149799 -1.195377" rpy="0 0 0"/>
-    <geometry>
-      <mesh filename="file://$(find r1d1_description)/meshes/arm_c4_1.stl" scale="0.001 0.001 0.001"/>
-    </geometry>
-    <material name="silver"/>
-  </visual>
-  <collision>
-    <origin xyz="-0.23574 0.149799 -1.195377" rpy="0 0 0"/>
-    <geometry>
-      <mesh filename="file://$(find r1d1_description)/meshes/arm_c4_1.stl" scale="0.001 0.001 0.001"/>
-    </geometry>
-  </collision>
-</link>
-<link name="arm_c5_1">
-  <inertial>
-    <origin xyz="0.027931367316718747 0.001141639371120412 -0.03694297864771845" rpy="0 0 0"/>
-    <mass value="0.7917902286710067"/>
-    <inertia ixx="0.000962" iyy="0.001203" izz="0.00093" ixy="6.1e-05" iyz="6.5e-05" ixz="-0.00023"/>
-  </inertial>
-  <visual>
-    <origin xyz="-0.404577 0.149799 -1.365964" rpy="0 0 0"/>
-    <geometry>
-      <mesh filename="file://$(find r1d1_description)/meshes/arm_c5_1.stl" scale="0.001 0.001 0.001"/>
-    </geometry>
-    <material name="silver"/>
-  </visual>
-  <collision>
-    <origin xyz="-0.404577 0.149799 -1.365964" rpy="0 0 0"/>
-    <geometry>
-      <mesh filename="file://$(find r1d1_description)/meshes/arm_c5_1.stl" scale="0.001 0.001 0.001"/>
-    </geometry>
-  </collision>
-</link>
-<link name="arm_c6_1">
-  <inertial>
-    <origin xyz="0.03182669751725131 -0.007873936279006344 0.03129187486567342" rpy="0 0 0"/>
-    <mass value="0.6685877298515001"/>
-    <inertia ixx="0.00076" iyy="0.000958" izz="0.000763" ixy="5e-06" iyz="5e-06" ixz="0.000157"/>
-  </inertial>
-  <visual>
-    <origin xyz="-0.475637 0.158915 -1.368144" rpy="0 0 0"/>
-    <geometry>
-      <mesh filename="file://$(find r1d1_description)/meshes/arm_c6_1.stl" scale="0.001 0.001 0.001"/>
-    </geometry>
-    <material name="silver"/>
-  </visual>
-  <collision>
-    <origin xyz="-0.475637 0.158915 -1.368144" rpy="0 0 0"/>
-    <geometry>
-      <mesh filename="file://$(find r1d1_description)/meshes/arm_c6_1.stl" scale="0.001 0.001 0.001"/>
-    </geometry>
-  </collision>
-</link>
-<link name="amr_c3_1">
-  <inertial>
-    <origin xyz="0.13969122062090347 -8.388348304855242e-08 0.05844792124625198" rpy="0 0 0"/>
-    <mass value="2.940490372828695"/>
-    <inertia ixx="0.021212" iyy="0.039248" izz="0.021088" ixy="0.0" iyz="0.0" ixz="-0.01706"/>
-  </inertial>
-  <visual>
-    <origin xyz="-0.038112 0.149799 -0.997027" rpy="0 0 0"/>
-    <geometry>
-      <mesh filename="file://$(find r1d1_description)/meshes/amr_c3_1.stl" scale="0.001 0.001 0.001"/>
-    </geometry>
-    <material name="silver"/>
-  </visual>
-  <collision>
-    <origin xyz="-0.038112 0.149799 -0.997027" rpy="0 0 0"/>
-    <geometry>
-      <mesh filename="file://$(find r1d1_description)/meshes/amr_c3_1.stl" scale="0.001 0.001 0.001"/>
-    </geometry>
-  </collision>
-</link>
-<link name="arm_c7_1">
-  <inertial>
-    <origin xyz="0.013946843385206464 3.245700232556992e-05 -0.01379788517027336" rpy="0 0 0"/>
-    <mass value="0.21151566499231975"/>
-    <inertia ixx="0.00014" iyy="0.000113" izz="0.00014" ixy="-0.0" iyz="-0.0" ixz="-2.7e-05"/>
-  </inertial>
-  <visual>
-    <origin xyz="-0.549936 0.167389 -1.361957" rpy="0 0 0"/>
-    <geometry>
-      <mesh filename="file://$(find r1d1_description)/meshes/arm_c7_1.stl" scale="0.001 0.001 0.001"/>
-    </geometry>
-    <material name="silver"/>
-  </visual>
-  <collision>
-    <origin xyz="-0.549936 0.167389 -1.361957" rpy="0 0 0"/>
-    <geometry>
-      <mesh filename="file://$(find r1d1_description)/meshes/arm_c7_1.stl" scale="0.001 0.001 0.001"/>
-    </geometry>
-  </collision>
-</link>
-<link name="gripper_base_1">
-  <inertial>
-    <origin xyz="0.050859725463711425 -2.1799271313072133e-07 -0.0506748564046926" rpy="0 0 0"/>
-    <mass value="0.7474580686995151"/>
-    <inertia ixx="0.001142" iyy="0.00191" izz="0.001145" ixy="4.3e-05" iyz="4.4e-05" ixz="0.000429"/>
-  </inertial>
-  <visual>
-    <origin xyz="-0.580397 0.167389 -1.331607" rpy="0 0 0"/>
-    <geometry>
-      <mesh filename="file://$(find r1d1_description)/meshes/gripper_base_1.stl" scale="0.001 0.001 0.001"/>
-    </geometry>
-    <material name="silver"/>
-  </visual>
-  <collision>
-    <origin xyz="-0.580397 0.167389 -1.331607" rpy="0 0 0"/>
-    <geometry>
-      <mesh filename="file://$(find r1d1_description)/meshes/gripper_base_1.stl" scale="0.001 0.001 0.001"/>
-    </geometry>
-  </collision>
-</link>
-<!--Removed rgbd camera code from here and added to rgbd_camera.xacro-->
-<!--Removed lidar_1 link code from here and added to lidar.xacro-->
-<joint name="left_wheel_joint" type="continuous">
-  <origin xyz="0.125905 0.011214 0.01" rpy="0 0 0"/>
-  <parent link="base_link"/>
-  <child link="left_wheel_1"/>
-  <axis xyz="-1.0 0.0 0.0"/>
-</joint>
-<joint name="right_wheel_joint" type="continuous">
-  <origin xyz="-0.125905 0.011214 0.01" rpy="0 0 0"/>
-  <parent link="base_link"/>
-  <child link="right_wheel_1"/>
-  <axis xyz="1.0 -0.0 0.0"/>
-</joint>
-<joint name="Rigid 7" type="fixed">
-  <origin xyz="0.0 0.0 0.0" rpy="0 0 0"/>
-  <parent link="base_link"/>
-  <child link="caster_1_1"/>
-</joint>
-<joint name="Rigid 21" type="fixed">
-  <origin xyz="0.0 0.0 0.28" rpy="0 0 0"/>
-  <parent link="base_link"/>
-  <child link="mount_v1_1"/>
-</joint>
-<joint name="Rigid 23" type="fixed">
-  <origin xyz="-0.300276 0.208406 2.495761" rpy="0 0 0"/>
-  <parent link="mount_v1_1"/>
-  <child link="vertical_v1_1"/>
-</joint>
-<joint name="Slider 29" type="prismatic">
-  <origin xyz="1.429463 0.07146 -0.432363" rpy="0 0 0"/>
-  <parent link="gripper_base_1"/>
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
File: r1d1_description/urdf/rgbd_camera.xacro (robot description, xacro)
@@ -1,51 +1,55 @@
 <?xml version="1.0"?>
-<robot xmlns:xacro="http://www.ros.org/wiki/xacro" >
-  <joint name="Rigid 45" type="fixed">
+<robot xmlns:xacro="http://www.ros.org/wiki/xacro">
+  <joint name="Rigid 45" type="revolute">
     <origin xyz="0.0 -0.117 0.0525" rpy="0 0 0"/>
     <parent link="screen_v1_1"/>
     <child link="camera_1"/>
+    <axis xyz="0 0 1"/>
+    <limit lower="0" upper="0" effort="0" velocity="0"/>
   </joint>
   <link name="camera_1">
     <inertial>
-        <origin xyz="6.1791840987637954e-15 -0.01000010951681022 -7.127631818093505e-14" rpy="0 0 0"/>
-        <mass value="0.05166258768470149"/>
-        <inertia ixx="3e-06" iyy="1.9e-05" izz="1.9e-05" ixy="-0.0" iyz="0.0" ixz="-0.0"/>
+      <origin xyz="6.1791840987637954e-15 -0.01000010951681022 -7.127631818093505e-14" rpy="0 0 0"/>
+      <mass value="0.05166258768470149"/>
+      <inertia ixx="3e-06" iyy="1.9e-05" izz="1.9e-05" ixy="-0.0" iyz="0.0" ixz="-0.0"/>
     </inertial>
     <visual>
-        <origin xyz="-0.0 0.031999 -1.8375" rpy="0 0 0"/>
-        <geometry>
+      <origin xyz="-0.0 0.031999 -1.8375" rpy="0 0 0"/>
+      <geometry>
         <mesh filename="file://$(find r1d1_description)/meshes/camera_1.stl" scale="0.001 0.001 0.001"/>
-        </geometry>
-        <material name="silver"/>
+      </geometry>
+      <material name="silver"/>
     </visual>
     <collision>
-        <origin xyz="-0.0 0.031999 -1.8375" rpy="0 0 0"/>
-        <geometry>
+      <origin xyz="-0.0 0.031999 -1.8375" rpy="0 0 0"/>
+      <geometry>
         <mesh filename="file://$(find r1d1_description)/meshes/camera_1.stl" scale="0.001 0.001 0.001"/>
-        </geometry>
+      </geometry>
     </collision>
   </link>
   <gazebo reference="camera_1">
-    <material>Gazebo/Red</material>
     <sensor name="rgbd_camera" type="rgbd_camera">
-        <camera>
-        <horizontal_fov>1.047</horizontal_fov>
+      <!--The pose here is a bit random so need to be adjusted-->
+      <pose>-0.0 -1.0 1.5 0 0 -1.5708</pose>
+      <camera>
+        <horizontal_fov>1.2</horizontal_fov>
         <image>
-            <width>600</width>
-            <height>400</height>
+          <width>640</width>
+          <height>480</height>
+          <format>BAYER_RGGB8</format>
         </image>
         <clip>
-            <near>0.1</near>
-            <far>100</far>
+          <near>0.02</near>
+          <far>10</far>
         </clip>
-        </camera>
-        <always_on>1</always_on>
-        <!--If running at good RTF then lower the update rate to 30 or so-->
-        <update_rate>1000</update_rate>
-        <visualize>true</visualize>
-        <topic>rgbd_camera</topic>
-        <plugin filename="ignition-gazebo-sensors-system" name="gz::sim::systems::Sensors">
-          <render_engine>ogre2</render_engine>
-        </plugin>
+      </camera>
+      <always_on>1</always_on>
+      <!--If running at good RTF then lower the update rate to 30 or so-->
+      <update_rate>10000</update_rate>
+      <visualize>true</visualize>
+      <topic>rgbd_camera</topic>
+      <plugin filename="ignition-gazebo-sensors-system" name="gz::sim::systems::Sensors">
+        <render_engine>ogre2</render_engine>
+      </plugin>
     </sensor>
   </gazebo>
