Commit message: added ignition controller code

File: r1d1_description/urdf/r1d1_m.urdf (robot description, URDF)
Before this commit: robot robot, 17 links, 16 joints
Links:
- removed link arm_base_link_1
- removed link base_footprint
- removed link c1_1
- removed link c2_1
- removed link c3_1
- removed link c4_1
- removed link forearm_Link_1
- removed link laser_frame
- removed link linear_1
- removed link shoulder_Link_1
- removed link upperarm_Link_1
- removed link wrist1_Link_1
- removed link wrist2_Link_1
- removed link wrist3_Link_1
- added link amr_c2_1, mass 0.8336850329541245; collision mesh filename=file:///home/ishan/OpenDroids_ws/install/r1d1_description/s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 scale=0.001 0.001 0.001; visual mesh filename=file:///home/ishan/OpenDroids_ws/install/r1d1_description/s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 scale=0.001 0.001 0.001
- added link amr_c3_1, mass 2.940490372828695; collision mesh filename=file:///home/ishan/OpenDroids_ws/install/r1d1_description/s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 scale=0.001 0.001 0.001; visual mesh filename=file:///home/ishan/OpenDroids_ws/install/r1d1_description/s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 scale=0.001 0.001 0.001
- added link arm_c1_1, mass 0.3077654114507175; collision mesh filename=file:///home/ishan/OpenDroids_ws/install/r1d1_description/s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 scale=0.001 0.001 0.001; visual mesh filename=file:///home/ishan/OpenDroids_ws/install/r1d1_description/s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 scale=0.001 0.001 0.001
- added link arm_c4_1, mass 1.9148915468217087; collision mesh filename=file:///home/ishan/OpenDroids_ws/install/r1d1_description/s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 scale=0.001 0.001 0.001; visual mesh filename=file:///home/ishan/OpenDroids_ws/install/r1d1_description/s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 scale=0.001 0.001 0.001
- added link arm_c5_1, mass 0.7917902286710067; collision mesh filename=file:///home/ishan/OpenDroids_ws/install/r1d1_description/s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 scale=0.001 0.001 0.001; visual mesh filename=file:///home/ishan/OpenDroids_ws/install/r1d1_description/s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 scale=0.001 0.001 0.001
- added link arm_c6_1, mass 0.6685877298515001; collision mesh filename=file:///home/ishan/OpenDroids_ws/install/r1d1_description/s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 scale=0.001 0.001 0.001; visual mesh filename=file:///home/ishan/OpenDroids_ws/install/r1d1_description/s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 scale=0.001 0.001 0.001
- added link arm_c7_1, mass 0.21151566499231975; collision mesh filename=file:///home/ishan/OpenDroids_ws/install/r1d1_description/s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 scale=0.001 0.001 0.001; visual mesh filename=file:///home/ishan/OpenDroids_ws/install/r1d1_description/s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 scale=0.001 0.001 0.001
- added link camera_1, mass 0.05166258768470149; collision mesh filename=file:///home/ishan/OpenDroids_ws/install/r1d1_description/s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 scale=0.001 0.001 0.001; visual mesh filename=file:///home/ishan/OpenDroids_ws/install/r1d1_description/s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 scale=0.001 0.001 0.001
- added link caster_1_1, mass 0.18492935556768103; collision mesh filename=file:///home/ishan/OpenDroids_ws/install/r1d1_description/s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 scale=0.001 0.001 0.001; visual mesh filename=file:///home/ishan/OpenDroids_ws/install/r1d1_description/s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 scale=0.001 0.001 0.001
- added link gripper_base_1, mass 0.7474580686995151; collision mesh filename=file:///home/ishan/OpenDroids_ws/install/r1d1_description/s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 scale=0.001 0.001 0.001; visual mesh filename=file:///home/ishan/OpenDroids_ws/install/r1d1_description/s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 scale=0.001 0.001 0.001
- added link gripper_finger2_1, mass 0.016384204166531253; collision mesh filename=file:///home/ishan/OpenDroids_ws/install/r1d1_description/s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 scale=0.001 0.001 0.001; visual mesh filename=file:///home/ishan/OpenDroids_ws/install/r1d1_description/s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 scale=0.001 0.001 0.001
- added link gripper_finger_1, mass 0.016384204166531253; collision mesh filename=file:///home/ishan/OpenDroids_ws/install/r1d1_description/s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 scale=0.001 0.001 0.001; visual mesh filename=file:///home/ishan/OpenDroids_ws/install/r1d1_description/s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 scale=0.001 0.001 0.001
- added link lidar_1, mass 0.6616194128460102; collision mesh filename=file:///home/ishan/OpenDroids_ws/install/r1d1_description/s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 scale=0.001 0.001 0.001; visual mesh filename=file:///home/ishan/OpenDroids_ws/install/r1d1_description/s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 scale=0.001 0.001 0.001
- added link mount_v1_1, mass 37.46152841680288; collision mesh filename=file:///home/ishan/OpenDroids_ws/install/r1d1_description/s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 scale=0.001 0.001 0.001; visual mesh filename=file:///home/ishan/OpenDroids_ws/install/r1d1_description/s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 scale=0.001 0.001 0.001
- added link screen_v1_1, mass 1.3238858059375562; collision mesh filename=file:///home/ishan/OpenDroids_ws/install/r1d1_description/s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 scale=0.001 0.001 0.001; visual mesh filename=file:///home/ishan/OpenDroids_ws/install/r1d1_description/s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 scale=0.001 0.001 0.001
- added link slider_1, mass 0.43604999999999994; collision mesh filename=file:///home/ishan/OpenDroids_ws/install/r1d1_description/s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 scale=0.001 0.001 0.001; visual mesh filename=file:///home/ishan/OpenDroids_ws/install/r1d1_description/s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 scale=0.001 0.001 0.001
- added link vertical_v1_1, mass 24.32699999999999; collision mesh filename=file:///home/ishan/OpenDroids_ws/install/r1d1_description/s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 scale=0.001 0.001 0.001; visual mesh filename=file:///home/ishan/OpenDroids_ws/install/r1d1_description/s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 scale=0.001 0.001 0.001
- link base_link: mass 55.61253674388458 -> 36.898914712235424; geometry collision mesh filename=file:///home/ishan/OpenDroids_ws/install/r1d1_description/s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 scale=0.001 0.001 0.001; visual mesh filename=file:///home/ishan/OpenDroids_ws/install/r1d1_description/s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 scale=0.001 0.001 0.001
- link left_wheel_1: mass 3.081377574152813 -> 1.2020197871482743; geometry collision mesh filename=file:///home/ishan/OpenDroids_ws/install/r1d1_description/s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 scale=0.001 0.001 0.001; visual mesh filename=file:///home/ishan/OpenDroids_ws/install/r1d1_description/s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 scale=0.001 0.001 0.001
- link right_wheel_1: mass 3.0813775741527913 -> 1.2020197871482743; geometry collision mesh filename=file:///home/ishan/OpenDroids_ws/install/r1d1_description/s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 scale=0.001 0.001 0.001; visual mesh filename=file:///home/ishan/OpenDroids_ws/install/r1d1_description/s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 scale=0.001 0.001 0.001
Joints:
- removed joint arm_fixed_joint
- removed joint base_footprint_joint
- removed joint castor_1
- removed joint castor_2
- removed joint castor_3
- removed joint castor_4
- removed joint forearm_joint
- removed joint laser_joint
- removed joint shoulder_joint
- removed joint slider
- removed joint upperarm_joint
- removed joint wrist_joint_1
- removed joint wrist_joint_2
- removed joint wrist_joint_3
- added joint Revolute 35: type continuous, parent arm_c1_1, child amr_c2_1, origin xyz=0.0 -0.0798 0.0 rpy=0 0 0, axis 0.0 -1.0 -0.0
- added joint Revolute 38: type continuous, parent amr_c3_1, child arm_c4_1, origin xyz=0.197628 0.0 0.19835 rpy=0 0 0, axis 0.708394 0.0 -0.705817
- added joint Revolute 39: type continuous, parent arm_c4_1, child arm_c5_1, origin xyz=0.168837 0.0 0.170587 rpy=0 0 0, axis -0.708394 -0.0 0.705817
- added joint Revolute 40: type continuous, parent arm_c5_1, child arm_c6_1, origin xyz=0.07106 -0.009116 0.00218 rpy=0 0 0, axis -0.695094 0.173648 -0.697632
- added joint Revolute 41: type continuous, parent amr_c2_1, child amr_c3_1, origin xyz=0.038112 -0.06 -0.037973 rpy=0 0 0, axis 0.708394 0.0 -0.705817
- added joint Revolute 42: type continuous, parent arm_c6_1, child arm_c7_1, origin xyz=0.074299 -0.008474 -0.006187 rpy=0 0 0, axis 0.708394 0.0 -0.705817
- added joint Rigid 21: type fixed, parent base_link, child mount_v1_1, origin xyz=0.0 0.0 0.28 rpy=0 0 0
- added joint Rigid 23: type fixed, parent mount_v1_1, child vertical_v1_1, origin xyz=-0.300276 0.208406 2.495761 rpy=0 0 0
- added joint Rigid 31: type fixed, parent vertical_v1_1, child screen_v1_1, origin xyz=0.300276 -0.123405 -0.990761 rpy=0 0 0
- added joint Rigid 34: type fixed, parent slider_1, child arm_c1_1, origin xyz=0.0 -0.005 0.0 rpy=0 0 0
- added joint Rigid 43: type fixed, parent arm_c7_1, child gripper_base_1, origin xyz=0.030461 0.0 -0.03035 rpy=0 0 0
- added joint Rigid 45: type revolute, parent screen_v1_1, child camera_1, origin xyz=0.0 -0.117 0.0525 rpy=0 0 0, axis 0 0 1, limit lower=0 upper=0 effort=0 velocity=0
- added joint Rigid 46: type fixed, parent base_link, child lidar_1, origin xyz=0.0 -0.123483 0.155 rpy=0 0 0
- added joint Rigid 7: type fixed, parent base_link, child caster_1_1, origin xyz=0.0 0.0 0.0 rpy=0 0 0
- added joint Slider 29: type prismatic, parent gripper_base_1, child gripper_finger_1, origin xyz=1.429463 0.07146 -0.432363 rpy=0 0 0, axis 0.695094 -0.173648 0.697632, limit lower=0.0055 upper=0.045 effort=100 velocity=100
- added joint Slider 30: type prismatic, parent gripper_base_1, child gripper_finger2_1, origin xyz=1.429463 0.07146 -0.432363 rpy=0 0 0, axis 0.695094 -0.173648 0.697632, limit lower=-0.04 upper=-0.0005 effort=100 velocity=100
- added joint Slider 33: type prismatic, parent vertical_v1_1, child slider_1, origin xyz=0.300276 -0.213405 -1.740761 rpy=0 0 0, axis 0.0 -0.0 1.0, limit lower=-0.64 upper=0.64 effort=100 velocity=100
- joint left_wheel_joint: axis -0.0 1.0 0.0 -> -1.0 0.0 0.0; origin xyz=0.0 0.105 0.085 rpy=0 0 0 -> xyz=0.125905 0.011214 0.01 rpy=0 0 0
- joint right_wheel_joint: axis 0.0 1.0 -0.0 -> 1.0 -0.0 0.0; origin xyz=0.0 -0.105 0.085 rpy=0 0 0 -> xyz=-0.125905 0.011214 0.01 rpy=0 0 0

File: r1d1_description/urdf/r1d1_m.xacro (robot description, xacro)
@@ -4,7 +4,137 @@
     <xacro:arg name="sim_mode" default="true"/>
     <xacro:include filename="$(find r1d1_description)/urdf/r1d1.xacro" />
-    <xacro:if value="$(arg use_ros2_control)">
-        <xacro:include filename="$(find r1d1_description)/urdf/ros2_control.xacro" />
+    <xacro:unless value="$(arg sim_mode)">
+        <ros2_control name="RealRobot" type="system">
+            <hardware>
+                <plugin>diffdrive_arduino/DiffDriveArduino</plugin>
+                <param name="left_wheel_name">left_wheel_joint</param>
+                <param name="right_wheel_name">right_wheel_joint</param>
+                <param name="loop_rate">30</param>
+                <param name="device">/dev/ttyUSB0</param>
+                <param name="baud_rate">57600</param>
+                <param name="timeout">1000</param>
+                <param name="enc_counts_per_rev">3436</param>
+            </hardware>
+            <joint name="left_wheel_joint">
+                <command_interface name="velocity">
+                    <param name="min">-10</param>
+                    <param name="max">10</param>
+                </command_interface>
+                <state_interface name="velocity"/>
+                <state_interface name="position"/>
+            </joint>
+            <joint name="right_wheel_joint">
+                <command_interface name="velocity">
+                    <param name="min">-10</param>
+                    <param name="max">10</param>
+                </command_interface>
+                <state_interface name="velocity"/>
+                <state_interface name="position"/>
+            </joint>
+        </ros2_control>
+    </xacro:unless>
+    <xacro:if value="$(arg sim_mode)">
+        <ros2_control name="IgnitionSystem" type="system">
+            <hardware>
+                <plugin>ign_ros2_control/IgnitionSystem</plugin>
+            </hardware>
+            <joint name="Slider 33">
+                <command_interface name="position"/>
+                <state_interface name="position">
+                    <param name="initial_value">0.3</param>
+                </state_interface>
+                <state_interface name="velocity"/>
+            </joint>
+            <joint name="Revolute 35">
+                <command_interface name="position">
+                </command_interface>
+                <state_interface name="position">
+                    <param name="initial_value">1.48</param>
+                </state_interface>
+                <state_interface name="velocity"/>
+                <state_interface name="effort"/>
+            </joint>
+            <joint name="Revolute 41">
+                <command_interface name="position">
+                </command_interface>
+                <state_interface name="position">
+                    <param name="initial_value">0.5</param>
+                </state_interface>
+                <state_interface name="velocity"/>
+                <state_interface name="effort"/>
+            </joint>
+            <joint name="Revolute 38">
+                <command_interface name="position">
+                </command_interface>
+                <state_interface name="position">
+                    <param name="initial_value">2.182</param>
+                </state_interface>
+                <state_interface name="velocity"/>
+                <state_interface name="effort"/>
+            </joint>
+            <joint name="Revolute 39">
+                <command_interface name="position">
+                </command_interface>
+                <state_interface name="position">
+                    <param name="initial_value">5.6</param>
+                </state_interface>
+                <state_interface name="velocity"/>
+                <state_interface name="effort"/>
+            </joint>
+            <joint name="Revolute 40">
+                <command_interface name="position">
+                </command_interface>
+                <state_interface name="position">
+                    <param name="initial_value">0.55</param>
+                </state_interface>
+                <state_interface name="velocity"/>
+                <state_interface name="effort"/>
+            </joint>
+            <joint name="Revolute 42">
+                <command_interface name="position">
+                </command_interface>
+                <state_interface name="position">
+                    <param name="initial_value">1.8</param>
+                </state_interface>
+                <state_interface name="velocity"/>
+                <state_interface name="effort"/>
+            </joint>
+            <joint name="Slider 29">
+                <command_interface name="position"/>
+                <state_interface name="position">
+                    <param name="initial_value">0.0081</param>
+                </state_interface>
+                <state_interface name="velocity"/>
+            </joint>
+            <joint name="Slider 30">
+                <command_interface name="position"/>
+                <state_interface name="position">
+                    <param name="initial_value">-0.0040</param>
+                </state_interface>
+                <state_interface name="velocity"/>
+            </joint>
+            <joint name="left_wheel_joint">
+                <command_interface name="velocity">
+                    <param name="min">-10</param>
+                    <param name="max">10</param>
+                </command_interface>
+                <state_interface name="position" />
+                <state_interface name="velocity" />
+            </joint>
+            <joint name="right_wheel_joint">
+                <command_interface name="velocity">
+                    <param name="min">-10</param>
+                    <param name="max">10</param>
+                </command_interface>
+                <state_interface name="velocity" />
+                <state_interface name="position" />
+            </joint>
+        </ros2_control>
     </xacro:if>
+    <gazebo>
+        <plugin filename="ign_ros2_control-system" name="ign_ros2_control::IgnitionROS2ControlPlugin">
+            <parameters>$(find r1d1_description)/config/r1d1.yaml</parameters>
+        </plugin>
+    </gazebo>
     <!-- <xacro:include filename="$(find r1d1_description)/urdf/gazebo_control.xacro" />     -->
     <!-- <xacro:include filename="$(find r1d1_description)/urdf/lidar.xacro" /> -->

File: r1d1_description/urdf/rgbd_camera.xacro (robot description, xacro)
@@ -41,5 +41,5 @@
         <clip>
           <near>0.02</near>
-          <far>10</far>
+          <far>8</far>
         </clip>
       </camera>
