Commit message: added ignition controller code

File: r1d1_description/urdf/ros2_control.xacro (robot description, xacro)
@@ -32,84 +32,84 @@
     </xacro:unless>
     <xacro:if value="$(arg sim_mode)">
-        <ros2_control name="GazeboSystem" type="system">
-        <hardware>
-            <plugin>gazebo_ros2_control/GazeboSystem</plugin>
-        </hardware>
-        <joint name="Slider 33">
-            <command_interface name="position"/>
-            <state_interface name="position">
-                <param name="initial_value">0.3</param>
-            </state_interface>
-            <state_interface name="velocity"/>
-        </joint>
-        <joint name="Revolute 35">
-            <command_interface name="position">
-            </command_interface>
-            <state_interface name="position">
-            <param name="initial_value">1.48</param>
-            </state_interface>
-            <state_interface name="velocity"/>
-            <state_interface name="effort"/>
-        </joint>
-        <joint name="Revolute 41">
-            <command_interface name="position">
-            </command_interface>
-            <state_interface name="position">
-            <param name="initial_value">0.5</param>
-            </state_interface>
-            <state_interface name="velocity"/>
-            <state_interface name="effort"/>
-        </joint>
-        <joint name="Revolute 38">
-            <command_interface name="position">
-            </command_interface>
-            <state_interface name="position">
-            <param name="initial_value">2.182</param>
-            </state_interface>
-            <state_interface name="velocity"/>
-            <state_interface name="effort"/>
-        </joint>
-        <joint name="Revolute 39">
-            <command_interface name="position">
-            </command_interface>
-            <state_interface name="position">
-            <param name="initial_value">5.6</param>
-            </state_interface>
-            <state_interface name="velocity"/>
-            <state_interface name="effort"/>
-        </joint>
-        <joint name="Revolute 40">
-            <command_interface name="position">
-            </command_interface>
-            <state_interface name="position">
-            <param name="initial_value">0.55</param>
-            </state_interface>
-            <state_interface name="velocity"/>
-            <state_interface name="effort"/>
-        </joint>
-        <joint name="Revolute 42">
-            <command_interface name="position">
-            </command_interface>
-            <state_interface name="position">
-            <param name="initial_value">1.8</param>
-            </state_interface>
-            <state_interface name="velocity"/>
-            <state_interface name="effort"/>
-        </joint>
-        <joint name="Slider 29">
-            <command_interface name="position"/>
-            <state_interface name="position">
-                <param name="initial_value">0.0081</param>
-            </state_interface>
-            <state_interface name="velocity"/>
-        </joint>
-        <joint name="Slider 30">
-            <command_interface name="position"/>
-            <state_interface name="position">
-                <param name="initial_value">-0.0040</param>
-            </state_interface>
-            <state_interface name="velocity"/>
-        </joint>
-        <joint name="left_wheel_joint">
+        <ros2_control name="IgnitionSystem" type="system">
+            <hardware>
+                <plugin>ign_ros2_control/IgnitionSystem</plugin>
+            </hardware>
+            <joint name="Slider 33">
+                <command_interface name="position"/>
+                <state_interface name="position">
+                    <param name="initial_value">0.3</param>
+                </state_interface>
+                <state_interface name="velocity"/>
+            </joint>
+            <joint name="Revolute 35">
+                <command_interface name="position">
+                </command_interface>
+                <state_interface name="position">
+                    <param name="initial_value">1.48</param>
+                </state_interface>
+                <state_interface name="velocity"/>
+                <state_interface name="effort"/>
+            </joint>
+            <joint name="Revolute 41">
+                <command_interface name="position">
+                </command_interface>
+                <state_interface name="position">
+                    <param name="initial_value">0.5</param>
+                </state_interface>
+                <state_interface name="velocity"/>
+                <state_interface name="effort"/>
+            </joint>
+            <joint name="Revolute 38">
+                <command_interface name="position">
+                </command_interface>
+                <state_interface name="position">
+                    <param name="initial_value">2.182</param>
+                </state_interface>
+                <state_interface name="velocity"/>
+                <state_interface name="effort"/>
+            </joint>
+            <joint name="Revolute 39">
+                <command_interface name="position">
+                </command_interface>
+                <state_interface name="position">
+                    <param name="initial_value">5.6</param>
+                </state_interface>
+                <state_interface name="velocity"/>
+                <state_interface name="effort"/>
+            </joint>
+            <joint name="Revolute 40">
+                <command_interface name="position">
+                </command_interface>
+                <state_interface name="position">
+                    <param name="initial_value">0.55</param>
+                </state_interface>
+                <state_interface name="velocity"/>
+                <state_interface name="effort"/>
+            </joint>
+            <joint name="Revolute 42">
+                <command_interface name="position">
+                </command_interface>
+                <state_interface name="position">
+                    <param name="initial_value">1.8</param>
+                </state_interface>
+                <state_interface name="velocity"/>
+                <state_interface name="effort"/>
+            </joint>
+            <joint name="Slider 29">
+                <command_interface name="position"/>
+                <state_interface name="position">
+                    <param name="initial_value">0.0081</param>
+                </state_interface>
+                <state_interface name="velocity"/>
+            </joint>
+            <joint name="Slider 30">
+                <command_interface name="position"/>
+                <state_interface name="position">
+                    <param name="initial_value">-0.0040</param>
+                </state_interface>
+                <state_interface name="velocity"/>
+            </joint>
+            <joint name="left_wheel_joint">
                 <command_interface name="velocity">
                     <param name="min">-10</param>
@@ -130,5 +130,5 @@
     </xacro:if>
     <gazebo>
-        <plugin filename="libgazebo_ros2_control.so" name="gazebo_ros2_control">
+        <plugin filename="ign_ros2_control-system" name="ign_ros2_control::IgnitionROS2ControlPlugin">
             <parameters>$(find r1d1_description)/config/r1d1.yaml</parameters>
         </plugin>
