Commit message: fix typos

File: r1d1_description/urdf/r1d1.xacro (robot description, xacro)
@@ -469,5 +469,5 @@
   <child link="screen_v1_1"/>
   <axis xyz="0 0 1"/>
-  <limit lower="0" upper="0" effor="0" velocity="0"/>
+  <limit lower="0" upper="0" effort="0" velocity="0"/>
 </joint>
 <joint name="Slider 33" type="prismatic">
@@ -529,5 +529,5 @@
   <child link="camera_1"/>
   <axis xyz="0 0 1"/>
-  <limit lower="0" upper="0" effor="0" velocity="0"/>
+  <limit lower="0" upper="0" effort="0" velocity="0"/>
 </joint>
 <joint name="Rigid 46" type="fixed">

Commit message: fix broken joint

File: r1d1_description/urdf/r1d1.xacro (robot description, xacro)
@@ -464,10 +464,8 @@
   <limit upper="-0.0005" lower="-0.04" effort="100" velocity="100"/>
 </joint>
-<joint name="Rigid 31" type="revolute">
+<joint name="Rigid 31" type="fixed">
   <origin xyz="0.300276 -0.123405 -0.990761" rpy="0 0 0"/>
   <parent link="vertical_v1_1"/>
   <child link="screen_v1_1"/>
-  <axis xyz="0 0 1"/>
-  <limit lower="0" upper="0" effort="0" velocity="0"/>
 </joint>
 <joint name="Slider 33" type="prismatic">

Commit message: GZ migrated sim hardware

File: r1d1_description/urdf/r1d1.xacro (robot description, xacro)
@@ -1,7 +1,25 @@
 <?xml version="1.0" ?>
 <robot name="r1d1" xmlns:xacro="http://www.ros.org/wiki/xacro">
-<xacro:include filename="$(find r1d1_description)/urdf/materials.xacro" />
-<xacro:include filename="$(find r1d1_description)/urdf/r1d1.trans" />
-<xacro:include filename="$(find r1d1_description)/urdf/r1d1.gazebo" />
+<material name="Red">
+  <color rgba="1 0 0 1"/>
+</material>
+<material name="Green">
+  <color rgba="0 1 0 1"/>
+</material>
+<material name="Blue">
+  <color rgba="0 0 1 1"/>
+</material>
+<material name="Yellow">
+  <color rgba="1 1 0 1"/>
+</material>
+<material name="Cyan">
+  <color rgba="0 1 1 1"/>
+</material>
+<material name="Magenta">
+  <color rgba="1 0 1 1"/>
+</material>
+<material name="White">
+  <color rgba="1 1 1 1"/>
+</material>
 <link name="base_link">
   <inertial>
@@ -13,12 +31,12 @@
     <origin xyz="0 0 0" rpy="0 0 0"/>
     <geometry>
-      <mesh filename="file://$(find r1d1_description)/meshes/base_link.stl" scale="0.001 0.001 0.001"/>
-    </geometry>
-    <material name="silver"/>
+      <mesh filename="file:///home/yugmil/ros2_ws/src/r1d1/r1d1_description/meshes/base_link.stl" scale="0.001 0.001 0.001"/>
+    </geometry>
+    <material name=""/>
   </visual>
   <collision>
     <origin xyz="0 0 0" rpy="0 0 0"/>
     <geometry>
-      <mesh filename="file://$(find r1d1_description)/meshes/base_link.stl" scale="0.001 0.001 0.001"/>
+      <mesh filename="file:///home/yugmil/ros2_ws/src/r1d1/r1d1_description/meshes/base_link.stl" scale="0.001 0.001 0.001"/>
     </geometry>
   </collision>
@@ -33,12 +51,12 @@
     <origin xyz="-0.125905 -0.011214 -0.01" rpy="0 0 0"/>
     <geometry>
-      <mesh filename="file://$(find r1d1_description)/meshes/left_wheel_1.stl" scale="0.001 0.001 0.001"/>
-    </geometry>
-    <material name="silver"/>
+      <mesh filename="file:///home/yugmil/ros2_ws/src/r1d1/r1d1_description/meshes/left_wheel_1.stl" scale="0.001 0.001 0.001"/>
+    </geometry>
+    <material name="White"/>
   </visual>
   <collision>
     <origin xyz="-0.125905 -0.011214 -0.01" rpy="0 0 0"/>
     <geometry>
-      <mesh filename="file://$(find r1d1_description)/meshes/left_wheel_1.stl" scale="0.001 0.001 0.001"/>
+      <mesh filename="file:///home/yugmil/ros2_ws/src/r1d1/r1d1_description/meshes/left_wheel_1.stl" scale="0.001 0.001 0.001"/>
     </geometry>
   </collision>
@@ -53,12 +71,12 @@
     <origin xyz="0.125905 -0.011214 -0.01" rpy="0 0 0"/>
     <geometry>
-      <mesh filename="file://$(find r1d1_description)/meshes/right_wheel_1.stl" scale="0.001 0.001 0.001"/>
-    </geometry>
-    <material name="silver"/>
+      <mesh filename="file:///home/yugmil/ros2_ws/src/r1d1/r1d1_description/meshes/right_wheel_1.stl" scale="0.001 0.001 0.001"/>
+    </geometry>
+    <material name="White"/>
   </visual>
   <collision>
     <origin xyz="0.125905 -0.011214 -0.01" rpy="0 0 0"/>
     <geometry>
-      <mesh filename="file://$(find r1d1_description)/meshes/right_wheel_1.stl" scale="0.001 0.001 0.001"/>
+      <mesh filename="file:///home/yugmil/ros2_ws/src/r1d1/r1d1_description/meshes/right_wheel_1.stl" scale="0.001 0.001 0.001"/>
     </geometry>
   </collision>
@@ -73,12 +91,12 @@
     <origin xyz="-0.0 -0.0 -0.0" rpy="0 0 0"/>
     <geometry>
-      <mesh filename="file://$(find r1d1_description)/meshes/caster_1_1.stl" scale="0.001 0.001 0.001"/>
-    </geometry>
-    <material name="silver"/>
+      <mesh filename="file:///home/yugmil/ros2_ws/src/r1d1/r1d1_description/meshes/caster_1_1.stl" scale="0.001 0.001 0.001"/>
+    </geometry>
+    <material name="White"/>
   </visual>
   <collision>
     <origin xyz="-0.0 -0.0 -0.0" rpy="0 0 0"/>
     <geometry>
-      <mesh filename="file://$(find r1d1_description)/meshes/caster_1_1.stl" scale="0.001 0.001 0.001"/>
+      <mesh filename="file:///home/yugmil/ros2_ws/src/r1d1/r1d1_description/meshes/caster_1_1.stl" scale="0.001 0.001 0.001"/>
     </geometry>
   </collision>
@@ -93,12 +111,12 @@
     <origin xyz="-0.0 -0.0 -0.28" rpy="0 0 0"/>
     <geometry>
-      <mesh filename="file://$(find r1d1_description)/meshes/mount_v1_1.stl" scale="0.001 0.001 0.001"/>
-    </geometry>
-    <material name="silver"/>
+      <mesh filename="file:///home/yugmil/ros2_ws/src/r1d1/r1d1_description/meshes/mount_v1_1.stl" scale="0.001 0.001 0.001"/>
+    </geometry>
+    <material name="White"/>
   </visual>
   <collision>
     <origin xyz="-0.0 -0.0 -0.28" rpy="0 0 0"/>
     <geometry>
-      <mesh filename="file://$(find r1d1_description)/meshes/mount_v1_1.stl" scale="0.001 0.001 0.001"/>
+      <mesh filename="file:///home/yugmil/ros2_ws/src/r1d1/r1d1_description/meshes/mount_v1_1.stl" scale="0.001 0.001 0.001"/>
     </geometry>
   </collision>
@@ -113,12 +131,12 @@
     <origin xyz="0.300276 -0.208406 -2.775761" rpy="0 0 0"/>
     <geometry>
-      <mesh filename="file://$(find r1d1_description)/meshes/vertical_v1_1.stl" scale="0.001 0.001 0.001"/>
-    </geometry>
-    <material name="silver"/>
+      <mesh filename="file:///home/yugmil/ros2_ws/src/r1d1/r1d1_description/meshes/vertical_v1_1.stl" scale="0.001 0.001 0.001"/>
+    </geometry>
+    <material name="White"/>
   </visual>
   <collision>
     <origin xyz="0.300276 -0.208406 -2.775761" rpy="0 0 0"/>
     <geometry>
-      <mesh filename="file://$(find r1d1_description)/meshes/vertical_v1_1.stl" scale="0.001 0.001 0.001"/>
+      <mesh filename="file:///home/yugmil/ros2_ws/src/r1d1/r1d1_description/meshes/vertical_v1_1.stl" scale="0.001 0.001 0.001"/>
     </geometry>
   </collision>
@@ -133,12 +151,12 @@
     <origin xyz="-2.00986 0.095929 -0.899244" rpy="0 0 0"/>
     <geometry>
-      <mesh filename="file://$(find r1d1_description)/meshes/gripper_finger_1.stl" scale="0.001 0.001 0.001"/>
-    </geometry>
-    <material name="silver"/>
+      <mesh filename="file:///home/yugmil/ros2_ws/src/r1d1/r1d1_description/meshes/gripper_finger_1.stl" scale="0.001 0.001 0.001"/>
+    </geometry>
+    <material name="White"/>
   </visual>
   <collision>
     <origin xyz="-2.00986 0.095929 -0.899244" rpy="0 0 0"/>
     <geometry>
-      <mesh filename="file://$(find r1d1_description)/meshes/gripper_finger_1.stl" scale="0.001 0.001 0.001"/>
+      <mesh filename="file:///home/yugmil/ros2_ws/src/r1d1/r1d1_description/meshes/gripper_finger_1.stl" scale="0.001 0.001 0.001"/>
     </geometry>
   </collision>
@@ -153,12 +171,12 @@
     <origin xyz="-2.00986 0.095929 -0.899244" rpy="0 0 0"/>
     <geometry>
-      <mesh filename="file://$(find r1d1_description)/meshes/gripper_finger2_1.stl" scale="0.001 0.001 0.001"/>
-    </geometry>
-    <material name="silver"/>
+      <mesh filename="file:///home/yugmil/ros2_ws/src/r1d1/r1d1_description/meshes/gripper_finger2_1.stl" scale="0.001 0.001 0.001"/>
+    </geometry>
+    <material name="White"/>
   </visual>
   <collision>
     <origin xyz="-2.00986 0.095929 -0.899244" rpy="0 0 0"/>
     <geometry>
-      <mesh filename="file://$(find r1d1_description)/meshes/gripper_finger2_1.stl" scale="0.001 0.001 0.001"/>
+      <mesh filename="file:///home/yugmil/ros2_ws/src/r1d1/r1d1_description/meshes/gripper_finger2_1.stl" scale="0.001 0.001 0.001"/>
     </geometry>
   </collision>
@@ -173,12 +191,12 @@
     <origin xyz="-0.0 -0.085001 -1.785" rpy="0 0 0"/>
     <geometry>
-      <mesh filename="file://$(find r1d1_description)/meshes/screen_v1_1.stl" scale="0.001 0.001 0.001"/>
-    </geometry>
-    <material name="silver"/>
+      <mesh filename="file:///home/yugmil/ros2_ws/src/r1d1/r1d1_description/meshes/screen_v1_1.stl" scale="0.001 0.001 0.001"/>
+    </geometry>
+    <material name="White"/>
   </visual>
   <collision>
     <origin xyz="-0.0 -0.085001 -1.785" rpy="0 0 0"/>
     <geometry>
-      <mesh filename="file://$(find r1d1_description)/meshes/screen_v1_1.stl" scale="0.001 0.001 0.001"/>
+      <mesh filename="file:///home/yugmil/ros2_ws/src/r1d1/r1d1_description/meshes/screen_v1_1.stl" scale="0.001 0.001 0.001"/>
     </geometry>
   </collision>
@@ -193,12 +211,12 @@
     <origin xyz="0.0 0.004999 -1.035" rpy="0 0 0"/>
     <geometry>
-      <mesh filename="file://$(find r1d1_description)/meshes/slider_1.stl" scale="0.001 0.001 0.001"/>
-    </geometry>
-    <material name="silver"/>
+      <mesh filename="file:///home/yugmil/ros2_ws/src/r1d1/r1d1_description/meshes/slider_1.stl" scale="0.001 0.001 0.001"/>
+    </geometry>
+    <material name="White"/>
   </visual>
   <collision>
     <origin xyz="0.0 0.004999 -1.035" rpy="0 0 0"/>
     <geometry>
-      <mesh filename="file://$(find r1d1_description)/meshes/slider_1.stl" scale="0.001 0.001 0.001"/>
+      <mesh filename="file:///home/yugmil/ros2_ws/src/r1d1/r1d1_description/meshes/slider_1.stl" scale="0.001 0.001 0.001"/>
     </geometry>
   </collision>
@@ -213,12 +231,12 @@
     <origin xyz="0.0 0.009999 -1.035" rpy="0 0 0"/>
     <geometry>
-      <mesh filename="file://$(find r1d1_description)/meshes/arm_c1_1.stl" scale="0.001 0.001 0.001"/>
-    </geometry>
-    <material name="silver"/>
+      <mesh filename="file:///home/yugmil/ros2_ws/src/r1d1/r1d1_description/meshes/arm_c1_1.stl" scale="0.001 0.001 0.001"/>
+    </geometry>
+    <material name="White"/>
   </visual>
   <collision>
     <origin xyz="0.0 0.009999 -1.035" rpy="0 0 0"/>
     <geometry>
-      <mesh filename="file://$(find r1d1_description)/meshes/arm_c1_1.stl" scale="0.001 0.001 0.001"/>
+      <mesh filename="file:///home/yugmil/ros2_ws/src/r1d1/r1d1_description/meshes/arm_c1_1.stl" scale="0.001 0.001 0.001"/>
     </geometry>
   </collision>
@@ -233,12 +251,12 @@
     <origin xyz="-0.0 0.089799 -1.035" rpy="0 0 0"/>
     <geometry>
-      <mesh filename="file://$(find r1d1_description)/meshes/amr_c2_1.stl" scale="0.001 0.001 0.001"/>
-    </geometry>
-    <material name="silver"/>
+      <mesh filename="file:///home/yugmil/ros2_ws/src/r1d1/r1d1_description/meshes/amr_c2_1.stl" scale="0.001 0.001 0.001"/>
+    </geometry>
+    <material name="White"/>
   </visual>
   <collision>
     <origin xyz="-0.0 0.089799 -1.035" rpy="0 0 0"/>
     <geometry>
-      <mesh filename="file://$(find r1d1_description)/meshes/amr_c2_1.stl" scale="0.001 0.001 0.001"/>
+      <mesh filename="file:///home/yugmil/ros2_ws/src/r1d1/r1d1_description/meshes/amr_c2_1.stl" scale="0.001 0.001 0.001"/>
     </geometry>
   </collision>
@@ -253,12 +271,12 @@
     <origin xyz="-0.23574 0.149799 -1.195377" rpy="0 0 0"/>
     <geometry>
-      <mesh filename="file://$(find r1d1_description)/meshes/arm_c4_1.stl" scale="0.001 0.001 0.001"/>
-    </geometry>
-    <material name="silver"/>
+      <mesh filename="file:///home/yugmil/ros2_ws/src/r1d1/r1d1_description/meshes/arm_c4_1.stl" scale="0.001 0.001 0.001"/>
+    </geometry>
+    <material name="White"/>
   </visual>
   <collision>
     <origin xyz="-0.23574 0.149799 -1.195377" rpy="0 0 0"/>
     <geometry>
-      <mesh filename="file://$(find r1d1_description)/meshes/arm_c4_1.stl" scale="0.001 0.001 0.001"/>
+      <mesh filename="file:///home/yugmil/ros2_ws/src/r1d1/r1d1_description/meshes/arm_c4_1.stl" scale="0.001 0.001 0.001"/>
     </geometry>
   </collision>
@@ -273,12 +291,12 @@
     <origin xyz="-0.404577 0.149799 -1.365964" rpy="0 0 0"/>
     <geometry>
-      <mesh filename="file://$(find r1d1_description)/meshes/arm_c5_1.stl" scale="0.001 0.001 0.001"/>
-    </geometry>
-    <material name="silver"/>
+      <mesh filename="file:///home/yugmil/ros2_ws/src/r1d1/r1d1_description/meshes/arm_c5_1.stl" scale="0.001 0.001 0.001"/>
+    </geometry>
+    <material name="White"/>
   </visual>
   <collision>
     <origin xyz="-0.404577 0.149799 -1.365964" rpy="0 0 0"/>
     <geometry>
-      <mesh filename="file://$(find r1d1_description)/meshes/arm_c5_1.stl" scale="0.001 0.001 0.001"/>
+      <mesh filename="file:///home/yugmil/ros2_ws/src/r1d1/r1d1_description/meshes/arm_c5_1.stl" scale="0.001 0.001 0.001"/>
     </geometry>
   </collision>
@@ -293,12 +311,12 @@
     <origin xyz="-0.475637 0.158915 -1.368144" rpy="0 0 0"/>
     <geometry>
-      <mesh filename="file://$(find r1d1_description)/meshes/arm_c6_1.stl" scale="0.001 0.001 0.001"/>
-    </geometry>
-    <material name="silver"/>
+      <mesh filename="file:///home/yugmil/ros2_ws/src/r1d1/r1d1_description/meshes/arm_c6_1.stl" scale="0.001 0.001 0.001"/>
+    </geometry>
+    <material name="White"/>
   </visual>
   <collision>
     <origin xyz="-0.475637 0.158915 -1.368144" rpy="0 0 0"/>
     <geometry>
-      <mesh filename="file://$(find r1d1_description)/meshes/arm_c6_1.stl" scale="0.001 0.001 0.001"/>
+      <mesh filename="file:///home/yugmil/ros2_ws/src/r1d1/r1d1_description/meshes/arm_c6_1.stl" scale="0.001 0.001 0.001"/>
     </geometry>
   </collision>
@@ -313,12 +331,12 @@
     <origin xyz="-0.038112 0.149799 -0.997027" rpy="0 0 0"/>
     <geometry>
-      <mesh filename="file://$(find r1d1_description)/meshes/amr_c3_1.stl" scale="0.001 0.001 0.001"/>
-    </geometry>
-    <material name="silver"/>
+      <mesh filename="file:///home/yugmil/ros2_ws/src/r1d1/r1d1_description/meshes/amr_c3_1.stl" scale="0.001 0.001 0.001"/>
+    </geometry>
+    <material name="White"/>
   </visual>
   <collision>
     <origin xyz="-0.038112 0.149799 -0.997027" rpy="0 0 0"/>
     <geometry>
-      <mesh filename="file://$(find r1d1_description)/meshes/amr_c3_1.stl" scale="0.001 0.001 0.001"/>
+      <mesh filename="file:///home/yugmil/ros2_ws/src/r1d1/r1d1_description/meshes/amr_c3_1.stl" scale="0.001 0.001 0.001"/>
     </geometry>
   </collision>
@@ -333,12 +351,12 @@
     <origin xyz="-0.549936 0.167389 -1.361957" rpy="0 0 0"/>
     <geometry>
-      <mesh filename="file://$(find r1d1_description)/meshes/arm_c7_1.stl" scale="0.001 0.001 0.001"/>
-    </geometry>
-    <material name="silver"/>
+      <mesh filename="file:///home/yugmil/ros2_ws/src/r1d1/r1d1_description/meshes/arm_c7_1.stl" scale="0.001 0.001 0.001"/>
+    </geometry>
+    <material name="White"/>
   </visual>
   <collision>
     <origin xyz="-0.549936 0.167389 -1.361957" rpy="0 0 0"/>
     <geometry>
-      <mesh filename="file://$(find r1d1_description)/meshes/arm_c7_1.stl" scale="0.001 0.001 0.001"/>
+      <mesh filename="file:///home/yugmil/ros2_ws/src/r1d1/r1d1_description/meshes/arm_c7_1.stl" scale="0.001 0.001 0.001"/>
     </geometry>
   </collision>
@@ -353,12 +371,12 @@
     <origin xyz="-0.580397 0.167389 -1.331607" rpy="0 0 0"/>
     <geometry>
-      <mesh filename="file://$(find r1d1_description)/meshes/gripper_base_1.stl" scale="0.001 0.001 0.001"/>
-    </geometry>
-    <material name="silver"/>
+      <mesh filename="file:///home/yugmil/ros2_ws/src/r1d1/r1d1_description/meshes/gripper_base_1.stl" scale="0.001 0.001 0.001"/>
+    </geometry>
+    <material name="White"/>
   </visual>
   <collision>
     <origin xyz="-0.580397 0.167389 -1.331607" rpy="0 0 0"/>
     <geometry>
-      <mesh filename="file://$(find r1d1_description)/meshes/gripper_base_1.stl" scale="0.001 0.001 0.001"/>
+      <mesh filename="file:///home/yugmil/ros2_ws/src/r1d1/r1d1_description/meshes/gripper_base_1.stl" scale="0.001 0.001 0.001"/>
     </geometry>
   </collision>
@@ -373,12 +391,12 @@
     <origin xyz="-0.0 0.031999 -1.8375" rpy="0 0 0"/>
     <geometry>
-      <mesh filename="file://$(find r1d1_description)/meshes/camera_1.stl" scale="0.001 0.001 0.001"/>
-    </geometry>
-    <material name="silver"/>
+      <mesh filename="file:///home/yugmil/ros2_ws/src/r1d1/r1d1_description/meshes/camera_1.stl" scale="0.001 0.001 0.001"/>
+    </geometry>
+    <material name="White"/>
   </visual>
   <collision>
     <origin xyz="-0.0 0.031999 -1.8375" rpy="0 0 0"/>
     <geometry>
-      <mesh filename="file://$(find r1d1_description)/meshes/camera_1.stl" scale="0.001 0.001 0.001"/>
+      <mesh filename="file:///home/yugmil/ros2_ws/src/r1d1/r1d1_description/meshes/camera_1.stl" scale="0.001 0.001 0.001"/>
     </geometry>
   </collision>
@@ -412,12 +430,12 @@
     <origin xyz="0.0 0.123483 -0.155" rpy="0 0 0"/>
     <geometry>
-      <mesh filename="file://$(find r1d1_description)/meshes/lidar_1.stl" scale="0.001 0.001 0.001"/>
-    </geometry>
-    <material name="silver"/>
+      <mesh filename="file:///home/yugmil/ros2_ws/src/r1d1/r1d1_description/meshes/lidar_1.stl" scale="0.001 0.001 0.001"/>
+    </geometry>
+    <material name="White"/>
   </visual>
   <collision>
     <origin xyz="0.0 0.123483 -0.155" rpy="0 0 0"/>
     <geometry>
-      <mesh filename="file://$(find r1d1_description)/meshes/lidar_1.stl" scale="0.001 0.001 0.001"/>
+      <mesh filename="file:///home/yugmil/ros2_ws/src/r1d1/r1d1_description/meshes/lidar_1.stl" scale="0.001 0.001 0.001"/>
     </geometry>
   </collision>
@@ -534,3 +552,30 @@
   <child link="lidar_1"/>
 </joint>
+<ros2_control name="GazeboSimSystem" type="system">
+  <hardware>
+      <plugin>gz_ros2_control/GazeboSimSystem</plugin>
+  </hardware>
+  <joint name="left_wheel_joint">
+      <command_interface name="velocity">
+          <param name="min">-10</param>
+          <param name="max">10</param>
+      </command_interface>
+      <state_interface name="position" />
+      <state_interface name="velocity" />
+  </joint>
+  <joint name="right_wheel_joint">
+      <command_interface name="velocity">
+          <param name="min">-10</param>
+          <param name="max">10</param>
+      </command_interface>
+      <state_interface name="velocity" />
+      <state_interface name="position" />
+  </joint>
+</ros2_control>
+<gazebo>
+  <plugin filename="gz_ros2_control-system" name="gz_ros2_control::GazeboSimROS2ControlPlugin">
+      <parameters>/home/yugmil/ros2_ws/src/r1d1/r1d1_description/config/r1d1.yaml</parameters>
+      <controller_manager_name>controller_manager</controller_manager_name>
+  </plugin>
+</gazebo>
 </robot>
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
File: r1d1_description/urdf/r1d1_m.xacro (robot description, xacro)
@@ -1,10 +1,6 @@
 <?xml version="1.0"?>
 <robot xmlns:xacro="http://www.ros.org/wiki/xacro"  name="robot">
-    <xacro:arg name="use_ros2_control" default="true"/>
-    <xacro:arg name="sim_mode" default="true"/>
-    <xacro:include filename="$(find r1d1_description)/urdf/r1d1.xacro" />
-    <xacro:if value="$(arg use_ros2_control)">
-        <xacro:include filename="$(find r1d1_description)/urdf/ros2_control.xacro" />
-    </xacro:if>
+    <xacro:include filename="r1d1.xacro"/>
+    <xacro:include filename="ros2_control.xacro"/>
     <!-- <xacro:include filename="$(find r1d1_description)/urdf/gazebo_control.xacro" />     -->
     <!-- <xacro:include filename="$(find r1d1_description)/urdf/lidar.xacro" /> -->
