Commit message: GZ migrated sim hardware

File: r1d1_description/urdf/ros2_control.xacro (robot description, xacro)
@@ -1,136 +1,105 @@
 <?xml version="1.0"?>
 <robot xmlns:xacro="http://www.ros.org/wiki/xacro">
-    <xacro:unless value="$(arg sim_mode)">
-        <ros2_control name="RealRobot" type="system">
-            <hardware>
-                <plugin>diffdrive_arduino/DiffDriveArduino</plugin>
-                <param name="left_wheel_name">left_wheel_joint</param>
-                <param name="right_wheel_name">right_wheel_joint</param>
-                <param name="loop_rate">30</param>
-                <param name="device">/dev/ttyUSB0</param>
-                <param name="baud_rate">57600</param>
-                <param name="timeout">1000</param>
-                <param name="enc_counts_per_rev">3436</param>
-            </hardware>
-            <joint name="left_wheel_joint">
-                <command_interface name="velocity">
-                    <param name="min">-10</param>
-                    <param name="max">10</param>
-                </command_interface>
-                <state_interface name="velocity"/>
-                <state_interface name="position"/>
-            </joint>
-            <joint name="right_wheel_joint">
-                <command_interface name="velocity">
-                    <param name="min">-10</param>
-                    <param name="max">10</param>
-                </command_interface>
-                <state_interface name="velocity"/>
-                <state_interface name="position"/>
-            </joint>
-        </ros2_control>
-    </xacro:unless>
-    <xacro:if value="$(arg sim_mode)">
-        <ros2_control name="GazeboSystem" type="system">
-        <hardware>
-            <plugin>gazebo_ros2_control/GazeboSystem</plugin>
-        </hardware>
-        <joint name="Slider 33">
-            <command_interface name="position"/>
-            <state_interface name="position">
-                <param name="initial_value">0.3</param>
-            </state_interface>
-            <state_interface name="velocity"/>
-        </joint>
-        <joint name="Revolute 35">
-            <command_interface name="position">
-            </command_interface>
-            <state_interface name="position">
-            <param name="initial_value">1.48</param>
-            </state_interface>
-            <state_interface name="velocity"/>
-            <state_interface name="effort"/>
-        </joint>
-        <joint name="Revolute 41">
-            <command_interface name="position">
-            </command_interface>
-            <state_interface name="position">
-            <param name="initial_value">0.5</param>
-            </state_interface>
-            <state_interface name="velocity"/>
-            <state_interface name="effort"/>
-        </joint>
-        <joint name="Revolute 38">
-            <command_interface name="position">
-            </command_interface>
-            <state_interface name="position">
-            <param name="initial_value">2.182</param>
-            </state_interface>
-            <state_interface name="velocity"/>
-            <state_interface name="effort"/>
-        </joint>
-        <joint name="Revolute 39">
-            <command_interface name="position">
-            </command_interface>
-            <state_interface name="position">
-            <param name="initial_value">5.6</param>
-            </state_interface>
-            <state_interface name="velocity"/>
-            <state_interface name="effort"/>
-        </joint>
-        <joint name="Revolute 40">
-            <command_interface name="position">
-            </command_interface>
-            <state_interface name="position">
-            <param name="initial_value">0.55</param>
-            </state_interface>
-            <state_interface name="velocity"/>
-            <state_interface name="effort"/>
-        </joint>
-        <joint name="Revolute 42">
-            <command_interface name="position">
-            </command_interface>
-            <state_interface name="position">
-            <param name="initial_value">1.8</param>
-            </state_interface>
-            <state_interface name="velocity"/>
-            <state_interface name="effort"/>
-        </joint>
-        <joint name="Slider 29">
-            <command_interface name="position"/>
-            <state_interface name="position">
-                <param name="initial_value">0.0081</param>
-            </state_interface>
-            <state_interface name="velocity"/>
-        </joint>
-        <joint name="Slider 30">
-            <command_interface name="position"/>
-            <state_interface name="position">
-                <param name="initial_value">-0.0040</param>
-            </state_interface>
-            <state_interface name="velocity"/>
-        </joint>
-        <joint name="left_wheel_joint">
-                <command_interface name="velocity">
-                    <param name="min">-10</param>
-                    <param name="max">10</param>
-                </command_interface>
-                <state_interface name="position" />
-                <state_interface name="velocity" />
-            </joint>
-            <joint name="right_wheel_joint">
-                <command_interface name="velocity">
-                    <param name="min">-10</param>
-                    <param name="max">10</param>
-                </command_interface>
-                <state_interface name="velocity" />
-                <state_interface name="position" />
-            </joint>
-        </ros2_control>
-    </xacro:if>
-    <gazebo>
-        <plugin filename="libgazebo_ros2_control.so" name="gazebo_ros2_control">
-            <parameters>$(find r1d1_description)/config/r1d1.yaml</parameters>
-        </plugin>
-    </gazebo>
+<ros2_control name="GazeboSimSystem" type="system">
+    <hardware>
+        <plugin>gz_ros2_control/GazeboSimSystem</plugin>
+    </hardware>
+    <joint name="Slider 33">
+        <command_interface name="position"/>
+        <state_interface name="position">
+            <param name="initial_value">0.3</param>
+        </state_interface>
+        <state_interface name="velocity"/>
+    </joint>
+    <joint name="Revolute 35">
+        <command_interface name="position">
+        </command_interface>
+        <state_interface name="position">
+        <param name="initial_value">1.48</param>
+        </state_interface>
+        <state_interface name="velocity"/>
+        <state_interface name="effort"/>
+    </joint>
+    <joint name="Revolute 41">
+        <command_interface name="position">
+        </command_interface>
+        <state_interface name="position">
+        <param name="initial_value">0.5</param>
+        </state_interface>
+        <state_interface name="velocity"/>
+        <state_interface name="effort"/>
+    </joint>
+    <joint name="Revolute 38">
+        <command_interface name="position">
+        </command_interface>
+        <state_interface name="position">
+        <param name="initial_value">2.182</param>
+        </state_interface>
+        <state_interface name="velocity"/>
+        <state_interface name="effort"/>
+    </joint>
+    <joint name="Revolute 39">
+        <command_interface name="position">
+        </command_interface>
+        <state_interface name="position">
+        <param name="initial_value">5.6</param>
+        </state_interface>
+        <state_interface name="velocity"/>
+        <state_interface name="effort"/>
+    </joint>
+    <joint name="Revolute 40">
+        <command_interface name="position">
+        </command_interface>
+        <state_interface name="position">
+        <param name="initial_value">0.55</param>
+        </state_interface>
+        <state_interface name="velocity"/>
+        <state_interface name="effort"/>
+    </joint>
+    <joint name="Revolute 42">
+        <command_interface name="position">
+        </command_interface>
+        <state_interface name="position">
+        <param name="initial_value">1.8</param>
+        </state_interface>
+        <state_interface name="velocity"/>
+        <state_interface name="effort"/>
+    </joint>
+    <joint name="Slider 29">
+        <command_interface name="position"/>
+        <state_interface name="position">
+            <param name="initial_value">0.0081</param>
+        </state_interface>
+        <state_interface name="velocity"/>
+    </joint>
+    <joint name="Slider 30">
+        <command_interface name="position"/>
+        <state_interface name="position">
+            <param name="initial_value">-0.0040</param>
+        </state_interface>
+        <state_interface name="velocity"/>
+    </joint>
+    <joint name="left_wheel_joint">
+        <command_interface name="velocity">
+            <param name="min">-10</param>
+            <param name="max">10</param>
+        </command_interface>
+        <state_interface name="position" />
+        <state_interface name="velocity" />
+    </joint>
+    <joint name="right_wheel_joint">
+        <command_interface name="velocity">
+            <param name="min">-10</param>
+            <param name="max">10</param>
+        </command_interface>
+        <state_interface name="velocity" />
+        <state_interface name="position" />
+    </joint>
+</ros2_control>
+<gazebo>
+    <plugin filename="libgazebo_ros2_control.so" name="gazebo_ros2_control">
+        <parameters>/home/yugmil/ros2_ws/src/r1d1/r1d1_description/config/r1d1.yaml</parameters>
+        <controller_manager_name>controller_manager</controller_manager_name>
+    </plugin>
+</gazebo>
 </robot>
