Commit message: debug

File: r1d1_description/urdf/r1d1.xacro (robot description, xacro)
@@ -31,5 +31,5 @@
     <origin xyz="0 0 0" rpy="0 0 0"/>
     <geometry>
-      <mesh filename="file:///home/yugmil/ros2_ws/src/r1d1/r1d1_description/meshes/base_link.stl" scale="0.001 0.001 0.001"/>
+      <mesh filename="file:($find r1d1_description)/meshes/base_link.stl" scale="0.001 0.001 0.001"/>
     </geometry>
     <material name=""/>
@@ -38,5 +38,5 @@
     <origin xyz="0 0 0" rpy="0 0 0"/>
     <geometry>
-      <mesh filename="file:///home/yugmil/ros2_ws/src/r1d1/r1d1_description/meshes/base_link.stl" scale="0.001 0.001 0.001"/>
+      <mesh filename="file:($find r1d1_description)/meshes/base_link.stl" scale="0.001 0.001 0.001"/>
     </geometry>
   </collision>
@@ -51,5 +51,5 @@
     <origin xyz="-0.125905 -0.011214 -0.01" rpy="0 0 0"/>
     <geometry>
-      <mesh filename="file:///home/yugmil/ros2_ws/src/r1d1/r1d1_description/meshes/left_wheel_1.stl" scale="0.001 0.001 0.001"/>
+      <mesh filename="file:($find r1d1_description)/meshes/left_wheel_1.stl" scale="0.001 0.001 0.001"/>
     </geometry>
     <material name="White"/>
@@ -58,5 +58,5 @@
     <origin xyz="-0.125905 -0.011214 -0.01" rpy="0 0 0"/>
     <geometry>
-      <mesh filename="file:///home/yugmil/ros2_ws/src/r1d1/r1d1_description/meshes/left_wheel_1.stl" scale="0.001 0.001 0.001"/>
+      <mesh filename="file:($find r1d1_description)/meshes/left_wheel_1.stl" scale="0.001 0.001 0.001"/>
     </geometry>
   </collision>
@@ -71,5 +71,5 @@
     <origin xyz="0.125905 -0.011214 -0.01" rpy="0 0 0"/>
     <geometry>
-      <mesh filename="file:///home/yugmil/ros2_ws/src/r1d1/r1d1_description/meshes/right_wheel_1.stl" scale="0.001 0.001 0.001"/>
+      <mesh filename="file:($find r1d1_description)/meshes/right_wheel_1.stl" scale="0.001 0.001 0.001"/>
     </geometry>
     <material name="White"/>
@@ -78,5 +78,5 @@
     <origin xyz="0.125905 -0.011214 -0.01" rpy="0 0 0"/>
     <geometry>
-      <mesh filename="file:///home/yugmil/ros2_ws/src/r1d1/r1d1_description/meshes/right_wheel_1.stl" scale="0.001 0.001 0.001"/>
+      <mesh filename="file:($find r1d1_description)/meshes/right_wheel_1.stl" scale="0.001 0.001 0.001"/>
     </geometry>
   </collision>
@@ -91,5 +91,5 @@
     <origin xyz="-0.0 -0.0 -0.0" rpy="0 0 0"/>
     <geometry>
-      <mesh filename="file:///home/yugmil/ros2_ws/src/r1d1/r1d1_description/meshes/caster_1_1.stl" scale="0.001 0.001 0.001"/>
+      <mesh filename="file:($find r1d1_description)/meshes/caster_1_1.stl" scale="0.001 0.001 0.001"/>
     </geometry>
     <material name="White"/>
@@ -98,5 +98,5 @@
     <origin xyz="-0.0 -0.0 -0.0" rpy="0 0 0"/>
     <geometry>
-      <mesh filename="file:///home/yugmil/ros2_ws/src/r1d1/r1d1_description/meshes/caster_1_1.stl" scale="0.001 0.001 0.001"/>
+      <mesh filename="file:($find r1d1_description)/meshes/caster_1_1.stl" scale="0.001 0.001 0.001"/>
     </geometry>
   </collision>
@@ -111,5 +111,5 @@
     <origin xyz="-0.0 -0.0 -0.28" rpy="0 0 0"/>
     <geometry>
-      <mesh filename="file:///home/yugmil/ros2_ws/src/r1d1/r1d1_description/meshes/mount_v1_1.stl" scale="0.001 0.001 0.001"/>
+      <mesh filename="file:($find r1d1_description)/meshes/mount_v1_1.stl" scale="0.001 0.001 0.001"/>
     </geometry>
     <material name="White"/>
@@ -118,5 +118,5 @@
     <origin xyz="-0.0 -0.0 -0.28" rpy="0 0 0"/>
     <geometry>
-      <mesh filename="file:///home/yugmil/ros2_ws/src/r1d1/r1d1_description/meshes/mount_v1_1.stl" scale="0.001 0.001 0.001"/>
+      <mesh filename="file:($find r1d1_description)/meshes/mount_v1_1.stl" scale="0.001 0.001 0.001"/>
     </geometry>
   </collision>
@@ -131,5 +131,5 @@
     <origin xyz="0.300276 -0.208406 -2.775761" rpy="0 0 0"/>
     <geometry>
-      <mesh filename="file:///home/yugmil/ros2_ws/src/r1d1/r1d1_description/meshes/vertical_v1_1.stl" scale="0.001 0.001 0.001"/>
+      <mesh filename="file:($find r1d1_description)/meshes/vertical_v1_1.stl" scale="0.001 0.001 0.001"/>
     </geometry>
     <material name="White"/>
@@ -138,5 +138,5 @@
     <origin xyz="0.300276 -0.208406 -2.775761" rpy="0 0 0"/>
     <geometry>
-      <mesh filename="file:///home/yugmil/ros2_ws/src/r1d1/r1d1_description/meshes/vertical_v1_1.stl" scale="0.001 0.001 0.001"/>
+      <mesh filename="file:($find r1d1_description)/meshes/vertical_v1_1.stl" scale="0.001 0.001 0.001"/>
     </geometry>
   </collision>
@@ -151,5 +151,5 @@
     <origin xyz="-2.00986 0.095929 -0.899244" rpy="0 0 0"/>
     <geometry>
-      <mesh filename="file:///home/yugmil/ros2_ws/src/r1d1/r1d1_description/meshes/gripper_finger_1.stl" scale="0.001 0.001 0.001"/>
+      <mesh filename="file:($find r1d1_description)/meshes/gripper_finger_1.stl" scale="0.001 0.001 0.001"/>
     </geometry>
     <material name="White"/>
@@ -158,5 +158,5 @@
     <origin xyz="-2.00986 0.095929 -0.899244" rpy="0 0 0"/>
     <geometry>
-      <mesh filename="file:///home/yugmil/ros2_ws/src/r1d1/r1d1_description/meshes/gripper_finger_1.stl" scale="0.001 0.001 0.001"/>
+      <mesh filename="file:($find r1d1_description)/meshes/gripper_finger_1.stl" scale="0.001 0.001 0.001"/>
     </geometry>
   </collision>
@@ -171,5 +171,5 @@
     <origin xyz="-2.00986 0.095929 -0.899244" rpy="0 0 0"/>
     <geometry>
-      <mesh filename="file:///home/yugmil/ros2_ws/src/r1d1/r1d1_description/meshes/gripper_finger2_1.stl" scale="0.001 0.001 0.001"/>
+      <mesh filename="file:($find r1d1_description)/meshes/gripper_finger2_1.stl" scale="0.001 0.001 0.001"/>
     </geometry>
     <material name="White"/>
@@ -178,5 +178,5 @@
     <origin xyz="-2.00986 0.095929 -0.899244" rpy="0 0 0"/>
     <geometry>
-      <mesh filename="file:///home/yugmil/ros2_ws/src/r1d1/r1d1_description/meshes/gripper_finger2_1.stl" scale="0.001 0.001 0.001"/>
+      <mesh filename="file:($find r1d1_description)/meshes/gripper_finger2_1.stl" scale="0.001 0.001 0.001"/>
     </geometry>
   </collision>
@@ -191,5 +191,5 @@
     <origin xyz="-0.0 -0.085001 -1.785" rpy="0 0 0"/>
     <geometry>
-      <mesh filename="file:///home/yugmil/ros2_ws/src/r1d1/r1d1_description/meshes/screen_v1_1.stl" scale="0.001 0.001 0.001"/>
+      <mesh filename="file:($find r1d1_description)/meshes/screen_v1_1.stl" scale="0.001 0.001 0.001"/>
     </geometry>
     <material name="White"/>
@@ -198,5 +198,5 @@
     <origin xyz="-0.0 -0.085001 -1.785" rpy="0 0 0"/>
     <geometry>
-      <mesh filename="file:///home/yugmil/ros2_ws/src/r1d1/r1d1_description/meshes/screen_v1_1.stl" scale="0.001 0.001 0.001"/>
+      <mesh filename="file:($find r1d1_description)/meshes/screen_v1_1.stl" scale="0.001 0.001 0.001"/>
     </geometry>
   </collision>
@@ -211,5 +211,5 @@
     <origin xyz="0.0 0.004999 -1.035" rpy="0 0 0"/>
     <geometry>
-      <mesh filename="file:///home/yugmil/ros2_ws/src/r1d1/r1d1_description/meshes/slider_1.stl" scale="0.001 0.001 0.001"/>
+      <mesh filename="file:($find r1d1_description)/meshes/slider_1.stl" scale="0.001 0.001 0.001"/>
     </geometry>
     <material name="White"/>
@@ -218,5 +218,5 @@
     <origin xyz="0.0 0.004999 -1.035" rpy="0 0 0"/>
     <geometry>
-      <mesh filename="file:///home/yugmil/ros2_ws/src/r1d1/r1d1_description/meshes/slider_1.stl" scale="0.001 0.001 0.001"/>
+      <mesh filename="file:($find r1d1_description)/meshes/slider_1.stl" scale="0.001 0.001 0.001"/>
     </geometry>
   </collision>
@@ -231,5 +231,5 @@
     <origin xyz="0.0 0.009999 -1.035" rpy="0 0 0"/>
     <geometry>
-      <mesh filename="file:///home/yugmil/ros2_ws/src/r1d1/r1d1_description/meshes/arm_c1_1.stl" scale="0.001 0.001 0.001"/>
+      <mesh filename="file:($find r1d1_description)/meshes/arm_c1_1.stl" scale="0.001 0.001 0.001"/>
     </geometry>
     <material name="White"/>
@@ -238,5 +238,5 @@
     <origin xyz="0.0 0.009999 -1.035" rpy="0 0 0"/>
     <geometry>
-      <mesh filename="file:///home/yugmil/ros2_ws/src/r1d1/r1d1_description/meshes/arm_c1_1.stl" scale="0.001 0.001 0.001"/>
+      <mesh filename="file:($find r1d1_description)/meshes/arm_c1_1.stl" scale="0.001 0.001 0.001"/>
     </geometry>
   </collision>
@@ -251,5 +251,5 @@
     <origin xyz="-0.0 0.089799 -1.035" rpy="0 0 0"/>
     <geometry>
-      <mesh filename="file:///home/yugmil/ros2_ws/src/r1d1/r1d1_description/meshes/amr_c2_1.stl" scale="0.001 0.001 0.001"/>
+      <mesh filename="file:($find r1d1_description)/meshes/amr_c2_1.stl" scale="0.001 0.001 0.001"/>
     </geometry>
     <material name="White"/>
@@ -258,5 +258,5 @@
     <origin xyz="-0.0 0.089799 -1.035" rpy="0 0 0"/>
     <geometry>
-      <mesh filename="file:///home/yugmil/ros2_ws/src/r1d1/r1d1_description/meshes/amr_c2_1.stl" scale="0.001 0.001 0.001"/>
+      <mesh filename="file:($find r1d1_description)/meshes/amr_c2_1.stl" scale="0.001 0.001 0.001"/>
     </geometry>
   </collision>
@@ -271,5 +271,5 @@
     <origin xyz="-0.23574 0.149799 -1.195377" rpy="0 0 0"/>
     <geometry>
-      <mesh filename="file:///home/yugmil/ros2_ws/src/r1d1/r1d1_description/meshes/arm_c4_1.stl" scale="0.001 0.001 0.001"/>
+      <mesh filename="file:($find r1d1_description)/meshes/arm_c4_1.stl" scale="0.001 0.001 0.001"/>
     </geometry>
     <material name="White"/>
@@ -278,5 +278,5 @@
     <origin xyz="-0.23574 0.149799 -1.195377" rpy="0 0 0"/>
     <geometry>
-      <mesh filename="file:///home/yugmil/ros2_ws/src/r1d1/r1d1_description/meshes/arm_c4_1.stl" scale="0.001 0.001 0.001"/>
+      <mesh filename="file:($find r1d1_description)/meshes/arm_c4_1.stl" scale="0.001 0.001 0.001"/>
     </geometry>
   </collision>
@@ -291,5 +291,5 @@
     <origin xyz="-0.404577 0.149799 -1.365964" rpy="0 0 0"/>
     <geometry>
-      <mesh filename="file:///home/yugmil/ros2_ws/src/r1d1/r1d1_description/meshes/arm_c5_1.stl" scale="0.001 0.001 0.001"/>
+      <mesh filename="file:($find r1d1_description)/meshes/arm_c5_1.stl" scale="0.001 0.001 0.001"/>
     </geometry>
     <material name="White"/>
@@ -298,5 +298,5 @@
     <origin xyz="-0.404577 0.149799 -1.365964" rpy="0 0 0"/>
     <geometry>
-      <mesh filename="file:///home/yugmil/ros2_ws/src/r1d1/r1d1_description/meshes/arm_c5_1.stl" scale="0.001 0.001 0.001"/>
+      <mesh filename="file:($find r1d1_description)/meshes/arm_c5_1.stl" scale="0.001 0.001 0.001"/>
     </geometry>
   </collision>
@@ -311,5 +311,5 @@
     <origin xyz="-0.475637 0.158915 -1.368144" rpy="0 0 0"/>
     <geometry>
-      <mesh filename="file:///home/yugmil/ros2_ws/src/r1d1/r1d1_description/meshes/arm_c6_1.stl" scale="0.001 0.001 0.001"/>
+      <mesh filename="file:($find r1d1_description)/meshes/arm_c6_1.stl" scale="0.001 0.001 0.001"/>
     </geometry>
     <material name="White"/>
@@ -318,5 +318,5 @@
     <origin xyz="-0.475637 0.158915 -1.368144" rpy="0 0 0"/>
     <geometry>
-      <mesh filename="file:///home/yugmil/ros2_ws/src/r1d1/r1d1_description/meshes/arm_c6_1.stl" scale="0.001 0.001 0.001"/>
+      <mesh filename="file:($find r1d1_description)/meshes/arm_c6_1.stl" scale="0.001 0.001 0.001"/>
     </geometry>
   </collision>
@@ -331,5 +331,5 @@
     <origin xyz="-0.038112 0.149799 -0.997027" rpy="0 0 0"/>
     <geometry>
-      <mesh filename="file:///home/yugmil/ros2_ws/src/r1d1/r1d1_description/meshes/amr_c3_1.stl" scale="0.001 0.001 0.001"/>
+      <mesh filename="file:($find r1d1_description)/meshes/amr_c3_1.stl" scale="0.001 0.001 0.001"/>
     </geometry>
     <material name="White"/>
@@ -338,5 +338,5 @@
     <origin xyz="-0.038112 0.149799 -0.997027" rpy="0 0 0"/>
     <geometry>
-      <mesh filename="file:///home/yugmil/ros2_ws/src/r1d1/r1d1_description/meshes/amr_c3_1.stl" scale="0.001 0.001 0.001"/>
+      <mesh filename="file:($find r1d1_description)/meshes/amr_c3_1.stl" scale="0.001 0.001 0.001"/>
     </geometry>
   </collision>
@@ -351,5 +351,5 @@
     <origin xyz="-0.549936 0.167389 -1.361957" rpy="0 0 0"/>
     <geometry>
-      <mesh filename="file:///home/yugmil/ros2_ws/src/r1d1/r1d1_description/meshes/arm_c7_1.stl" scale="0.001 0.001 0.001"/>
+      <mesh filename="file:($find r1d1_description)/meshes/arm_c7_1.stl" scale="0.001 0.001 0.001"/>
     </geometry>
     <material name="White"/>
@@ -358,5 +358,5 @@
     <origin xyz="-0.549936 0.167389 -1.361957" rpy="0 0 0"/>
     <geometry>
-      <mesh filename="file:///home/yugmil/ros2_ws/src/r1d1/r1d1_description/meshes/arm_c7_1.stl" scale="0.001 0.001 0.001"/>
+      <mesh filename="file:($find r1d1_description)/meshes/arm_c7_1.stl" scale="0.001 0.001 0.001"/>
     </geometry>
   </collision>
@@ -371,5 +371,5 @@
     <origin xyz="-0.580397 0.167389 -1.331607" rpy="0 0 0"/>
     <geometry>
-      <mesh filename="file:///home/yugmil/ros2_ws/src/r1d1/r1d1_description/meshes/gripper_base_1.stl" scale="0.001 0.001 0.001"/>
+      <mesh filename="file:($find r1d1_description)/meshes/gripper_base_1.stl" scale="0.001 0.001 0.001"/>
     </geometry>
     <material name="White"/>
@@ -378,5 +378,5 @@
     <origin xyz="-0.580397 0.167389 -1.331607" rpy="0 0 0"/>
     <geometry>
-      <mesh filename="file:///home/yugmil/ros2_ws/src/r1d1/r1d1_description/meshes/gripper_base_1.stl" scale="0.001 0.001 0.001"/>
+      <mesh filename="file:($find r1d1_description)/meshes/gripper_base_1.stl" scale="0.001 0.001 0.001"/>
     </geometry>
   </collision>
@@ -391,5 +391,5 @@
     <origin xyz="-0.0 0.031999 -1.8375" rpy="0 0 0"/>
     <geometry>
-      <mesh filename="file:///home/yugmil/ros2_ws/src/r1d1/r1d1_description/meshes/camera_1.stl" scale="0.001 0.001 0.001"/>
+      <mesh filename="file:($find r1d1_description)/meshes/camera_1.stl" scale="0.001 0.001 0.001"/>
     </geometry>
     <material name="White"/>
@@ -398,5 +398,5 @@
     <origin xyz="-0.0 0.031999 -1.8375" rpy="0 0 0"/>
     <geometry>
-      <mesh filename="file:///home/yugmil/ros2_ws/src/r1d1/r1d1_description/meshes/camera_1.stl" scale="0.001 0.001 0.001"/>
+      <mesh filename="file:($find r1d1_description)/meshes/camera_1.stl" scale="0.001 0.001 0.001"/>
     </geometry>
   </collision>
@@ -430,5 +430,5 @@
     <origin xyz="0.0 0.123483 -0.155" rpy="0 0 0"/>
     <geometry>
-      <mesh filename="file:///home/yugmil/ros2_ws/src/r1d1/r1d1_description/meshes/lidar_1.stl" scale="0.001 0.001 0.001"/>
+      <mesh filename="file:($find r1d1_description)/meshes/lidar_1.stl" scale="0.001 0.001 0.001"/>
     </geometry>
     <material name="White"/>
@@ -437,5 +437,5 @@
     <origin xyz="0.0 0.123483 -0.155" rpy="0 0 0"/>
     <geometry>
-      <mesh filename="file:///home/yugmil/ros2_ws/src/r1d1/r1d1_description/meshes/lidar_1.stl" scale="0.001 0.001 0.001"/>
+      <mesh filename="file:($find r1d1_description)/meshes/lidar_1.stl" scale="0.001 0.001 0.001"/>
     </geometry>
   </collision>
